File: decon_output.kicad_sch (KiCad schematic)
At the start: 144 parts, among them J10 Conn_01x02, J11 Conn_01x02, J12 Conn_01x02, J13 Conn_01x02, J14 Conn_01x02, J15 Conn_01x02, J16 Conn_01x02, J17 Conn_01x02, J18 Conn_01x02, J19 Conn_01x02, J20 Conn_01x02, J5 Conn_01x02, J6 Conn_01x02, J7 Conn_01x02, J8 Conn_01x02, J9 Conn_01x02, K10 G5NB, K11 G5NB, K12 G5NB, K13 G5NB, K14 G5NB, K15 G5NB, K16 G5NB, K17 G5NB, K18 G5NB, K19 G5NB, K20 G5NB, K5 G5NB, K6 G5NB, K7 G5NB, K8 G5NB, K9 G5NB, Q10 MMBT2222A, Q11 MMBT2222A, Q12 MMBT2222A, Q13 MMBT2222A, Q14 MMBT2222A, Q15 MMBT2222A, Q16 MMBT2222A, Q17 MMBT2222A, Q18 MMBT2222A, Q19 MMBT2222A, Q20 MMBT2222A, Q5 MMBT2222A, Q6 MMBT2222A, Q7 MMBT2222A, Q8 MMBT2222A, Q9 MMBT2222A, U10 LTV-817S, U11 LTV-817S, U12 LTV-817S, U13 LTV-817S, U14 LTV-817S, U15 LTV-817S, U16 LTV-817S, U17 LTV-817S, U18 LTV-817S, U19 LTV-817S, U20 LTV-817S, U21 LTV-817S, U6 LTV-817S, U7 LTV-817S, U8 LTV-817S, U9 LTV-817S

Commit message: modified:   DECON_Ctrl_Panel.kicad_pcb 	modified:   DECON_Ctrl_Panel.kicad_prl 	new file:   MCU_pins.xlsx 	new file:   Son_KiCad_lib/Son_KiCad_lib.bak 	new file:   Son_KiCad_lib/Son_KiCad_lib.kicad_sym 	new file:   Son_KiCad_lib/Son_KiCad_lib.pretty/URB2405YMD-10WR3.kicad_mod 	modified:   decon_input.kicad_sch 	modified:   decon_mcu.kicad_sch 	modified:   decon_output.kicad_sch 	modified:   decon_power.kicad_sch 	new file:   fp-lib-table 	new file:   sym-lib-table
Parts:
- removed C10, C11, C12, C13, C14, C15, C16, C18, C19, C20, C5, C6, C7, C8, C9: 104, Capacitor_SMD:C_0805_2012Metric, symbol Device:C
- removed D10, D11, D12, D17, D18, D19, D20, D25, D26, D27, D28, D34, D35, D36, D9: LED, LED_SMD:LED_0805_2012Metric, symbol Device:LED
- removed D13, D14, D15, D16, D21, D22, D23, D24, D29, D30, D31, D32, D38, D39, D40: 1N4148W, Diode_SMD:D_SOD-123, symbol Diode:1N4148W
- removed J10, J11, J12, J13, J14, J15, J16, J17, J18, J19, J20, J5, J6, J7, J8, J9: Conn_01x02, TerminalBlock_Phoenix:TerminalBlock_Phoenix_MKDS-1-2-3.81_1x02_P3.81mm_Horizontal, symbol Connector_Generic:Conn_01x02
- removed K10, K11, K12, K13, K14, K15, K16, K18, K19, K20, K5, K6, K7, K8, K9: G5NB, Relay_THT:Relay_SPST_Omron_G5NB, symbol Relay:G5NB
- removed Q10, Q11, Q12, Q13, Q14, Q15, Q16, Q18, Q19, Q20, Q5, Q6, Q7, Q8, Q9: MMBT2222A, Package_TO_SOT_SMD:SOT-23-3, symbol Transistor_BJT:MMBT2222A
- removed R10, R11, R12, R17, R18, R19, R20, R25, R26, R27, R28, R34, R35, R36, R9: 1K, Resistor_SMD:R_0805_2012Metric, symbol Device:R
- removed R13, R14, R15, R16, R21, R22, R23, R24, R29, R30, R31, R32, R38, R39, R40: 510, Resistor_SMD:R_0805_2012Metric, symbol Device:R
- removed U10, U11, U12, U13, U14, U15, U16, U17, U19, U20, U21, U6, U7, U8, U9: LTV-817S, Package_DIP:SMDIP-4_W9.53mm, symbol Isolator:LTV-817S
- added J24: Conn_01x10, Connector_Phoenix_MC:PhoenixContact_MC_1,5_10-G-3.81_1x10_P3.81mm_Horizontal, symbol Connector_Generic:Conn_01x10
Connections:
- net 24V is gone; now on net VBAT: D37.1 (K), K17.A1, U18.4
- net RELAY_0: now reaches C17.1, K17.13
- net MCU_GPIO renamed MCU_RL0
- new net GND_VBAT: J24.1 (Pin_1), J24.10 (Pin_10)
- new net LED_1: J24.2 (Pin_2)
- new net LED_2: J24.3 (Pin_3)
- new net LED_3: J24.4 (Pin_4)
- new net LED_4: J24.5 (Pin_5)
- new net LED_5: J24.6 (Pin_6)
- new net LED_6: J24.7 (Pin_7)
- new net LED_7: J24.8 (Pin_8)
- new net LED_8: J24.9 (Pin_9)

Commit message: modified:   DECON_Ctrl_Panel.kicad_sch
Parts:
- added C10, C11, C12, C13, C14, C15, C16, C18, C19, C20, C21, C22, C23, C8, C9: 104, Capacitor_SMD:C_0805_2012Metric, symbol Device:C
- added D10, D11, D14, D15, D18, D19, D22, D23, D26, D27, D3, D30, D31, D6, D7: 1N4148W, Diode_SMD:D_SOD-123, symbol Diode:1N4148W
- added D12, D13, D16, D17, D2, D20, D21, D24, D25, D28, D29, D4, D5, D8, D9: LED, LED_SMD:LED_0805_2012Metric, symbol Device:LED
- added K1, K10, K11, K12, K13, K14, K15, K2, K3, K4, K5, K6, K7, K8, K9: G5NB, Relay_THT:Relay_SPST_Omron_G5NB, symbol Relay:G5NB
- added Q1, Q10, Q11, Q12, Q13, Q14, Q15, Q2, Q3, Q4, Q5, Q6, Q7, Q8, Q9: MMBT2222A, Package_TO_SOT_SMD:SOT-23-3, symbol Transistor_BJT:MMBT2222A
- added R10, R11, R14, R15, R18, R19, R22, R23, R26, R27, R3, R30, R31, R6, R7: 510, Resistor_SMD:R_0805_2012Metric, symbol Device:R
- added R12, R13, R16, R17, R2, R20, R21, R24, R25, R28, R29, R4, R5, R8, R9: 1K, Resistor_SMD:R_0805_2012Metric, symbol Device:R
- added U10, U11, U12, U13, U14, U15, U16, U17, U19, U20, U5, U6, U7, U8, U9: LTV-817S, Package_DIP:SMDIP-4_W9.53mm, symbol Isolator:LTV-817S
Connections:
- net GND_24V is gone; now on net GND_VBAT: C17.2, Q17.2 (E)
- net 3.3V: now also R12.1, R13.1, R16.1, R17.1, R2.1, R20.1, R21.1, R24.1, R25.1, R28.1, R29.1, R4.1, R5.1, R8.1, R9.1
- net GND_VBAT: now also C10.2, C11.2, C12.2, C13.2, C14.2, C15.2, C16.2, C18.2, C19.2, C20.2, C21.2, C22.2, C23.2, C8.2, C9.2, Q1.2 (E), Q10.2 (E), Q11.2 (E), Q12.2 (E), Q13.2 (E), Q14.2 (E), Q15.2 (E), Q2.2 (E), Q3.2 (E), Q4.2 (E), Q5.2 (E), Q6.2 (E), Q7.2 (E), Q8.2 (E), Q9.2 (E)
- net VBAT: now also D10.1 (K), D11.1 (K), D14.1 (K), D15.1 (K), D18.1 (K), D19.1 (K), D22.1 (K), D23.1 (K), D26.1 (K), D27.1 (K), D3.1 (K), D30.1 (K), D31.1 (K), D6.1 (K), D7.1 (K), K1.14, K1.A1, K10.14, K10.A1, K11.14, K11.A1, K12.14, K12.A1, K13.14, K13.A1, K14.14, K14.A1, K15.14, K15.A1, K2.14, K2.A1, K3.14, K3.A1, K4.14, K4.A1, K5.14, K5.A1, K6.14, K6.A1, K7.14, K7.A1, K8.14, K8.A1, K9.14, K9.A1, U10.4, U11.4, U12.4, U13.4, U14.4, U15.4, U16.4, U17.4, U19.4, U20.4, U5.4, U6.4, U7.4, U8.4, U9.4
- new net: R4.2, U6.1
- new net: D2.2 (A), U5.2
- new net: R2.2, U5.1
- new net: D10.2 (A), K4.A2, Q4.3 (C)
- new net: D14.2 (A), K6.A2, Q6.3 (C)
- new net: R5.2, U7.1
- new net: D5.2 (A), U7.2
- new net: R7.1, U7.3
- new net: D21.2 (A), U15.2
- new net: R12.2, U10.1
- new net: D12.2 (A), U10.2
- new net: R14.1, U10.3
- new net: R18.1, U12.3
- new net: Q8.1 (B), R18.2
- new net: Q13.1 (B), R27.2
- new net: D27.2 (A), K13.A2, Q13.3 (C)
- new net: R3.1, U5.3
- new net: Q1.1 (B), R3.2
- new net: D24.2 (A), U16.2
- new net: D6.2 (A), K2.A2, Q2.3 (C)
- new net: R8.2, U8.1
- new net: D26.2 (A), K12.A2, Q12.3 (C)
- new net: R13.2, U11.1
- new net: D15.2 (A), K7.A2, Q7.3 (C)
- new net: R11.1, U9.3
- new net: Q5.1 (B), R11.2
- new net: D3.2 (A), K1.A2, Q1.3 (C)
- new net: D7.2 (A), K3.A2, Q3.3 (C)
- new net: R29.2, U20.1
- new net: D29.2 (A), U20.2
- new net: R31.1, U20.3
- new net: Q4.1 (B), R10.2
- new net: R9.2, U9.1
- new net: D31.2 (A), K15.A2, Q15.3 (C)
- new net: R15.1, U11.3
- new net: Q7.1 (B), R15.2
- new net: Q2.1 (B), R6.2
- new net: D23.2 (A), K11.A2, Q11.3 (C)
- new net: R25.2, U17.1
- new net: D25.2 (A), U17.2
- new net: R27.1, U17.3
- new net: D28.2 (A), U19.2
- new net: R24.2, U16.1
- new net: R26.1, U16.3
- new net: Q10.1 (B), R22.2
- new net: D22.2 (A), K10.A2, Q10.3 (C)
- new net: R21.2, U15.1
- new net: R23.1, U15.3
- new net: R20.2, U14.1
- new net: D8.2 (A), U8.2
- new net: D16.2 (A), U12.2
- new net: Q3.1 (B), R7.2
- new net: D11.2 (A), K5.A2, Q5.3 (C)
- new net: D18.2 (A), K8.A2, Q8.3 (C)
- new net: R30.1, U19.3
- new net: Q14.1 (B), R30.2
- new net: Q12.1 (B), R26.2
- new net: D30.2 (A), K14.A2, Q14.3 (C)
- new net: Q11.1 (B), R23.2
- new net: D4.2 (A), U6.2
- new net: R6.1, U6.3
- new net: D13.2 (A), U11.2
- new net: Q9.1 (B), R19.2
- new net: D19.2 (A), K9.A2, Q9.3 (C)
- new net: R17.2, U13.1
- new net: D17.2 (A), U13.2
- new net: R19.1, U13.3
- new net: Q15.1 (B), R31.2
- new net: D9.2 (A), U9.2
- new net: D20.2 (A), U14.2
- new net: R28.2, U19.1
- new net: Q6.1 (B), R14.2
- new net: R22.1, U14.3
- new net: R16.2, U12.1
- new net: R10.1, U8.3
- new net MCU_RL1: D2.1 (K)
- new net MCU_RL10: D24.1 (K)
- new net MCU_RL11: D25.1 (K)
- new net MCU_RL12: D12.1 (K)
- new net MCU_RL13: D13.1 (K)
- new net MCU_RL14: D28.1 (K)
- new net MCU_RL15: D29.1 (K)
- new net MCU_RL2: D16.1 (K)
- new net MCU_RL3: D17.1 (K)
- new net MCU_RL4: D4.1 (K)
- new net MCU_RL5: D5.1 (K)
- new net MCU_RL6: D20.1 (K)
- new net MCU_RL7: D21.1 (K)
- new net MCU_RL8: D8.1 (K)
- new net MCU_RL9: D9.1 (K)
- new net RELAY_1: C8.1, K1.13
- new net RELAY_10: C20.1, K12.13
- new net RELAY_11: C21.1, K13.13
- new net RELAY_12: C13.1, K6.13
- new net RELAY_13: C14.1, K7.13
- new net RELAY_14: C22.1, K14.13
- new net RELAY_15: C23.1, K15.13
- new net RELAY_2: C15.1, K8.13
- new net RELAY_3: C16.1, K9.13
- new net RELAY_4: C9.1, K2.13
- new net RELAY_5: C10.1, K3.13
- new net RELAY_6: C18.1, K10.13
- new net RELAY_7: C19.1, K11.13
- new net RELAY_8: C11.1, K4.13
- new net RELAY_9: C12.1, K5.13
