File: DECON_Ctrl_Panel.kicad_pcb (KiCad board)
At the start: 2 copper layers, 150 x 90 mm, 24 parts, among them J2 Conn_01x02, K1 G5NB, Q1 MMBT2222A, U1 LTV-817S

Commit message: modified:   DECON_Ctrl_Panel.kicad_pcb 	modified:   DECON_Ctrl_Panel.kicad_prl 	new file:   MCU_pins.xlsx 	new file:   Son_KiCad_lib/Son_KiCad_lib.bak 	new file:   Son_KiCad_lib/Son_KiCad_lib.kicad_sym 	new file:   Son_KiCad_lib/Son_KiCad_lib.pretty/URB2405YMD-10WR3.kicad_mod 	modified:   decon_input.kicad_sch 	modified:   decon_mcu.kicad_sch 	modified:   decon_output.kicad_sch 	modified:   decon_power.kicad_sch 	new file:   fp-lib-table 	new file:   sym-lib-table
Parts:
- removed C1 (x2): 104, Capacitor_SMD:C_0805_2012Metric
- removed D1 (x2): LED, LED_SMD:LED_0805_2012Metric
- removed D2 (x2): 1N4148W, Diode_SMD:D_SOD-123
- removed J2 (x2): Conn_01x02, TerminalBlock_Phoenix:TerminalBlock_Phoenix_MKDS-1-2-3.81_1x02_P3.81mm_Horizontal
- removed K1 (x2): G5NB, Relay_THT:Relay_SPST_Omron_G5NB
- removed Q1 (x2): MMBT2222A, Package_TO_SOT_SMD:SOT-23-3
- removed R1 (x2): 1K, Resistor_SMD:R_0805_2012Metric
- removed R2 (x2): 510, Resistor_SMD:R_0805_2012Metric
- removed REF** (x6): TerminalBlock_Phoenix_MKDS-1-10-3.81_1x10_P3.81mm_Horizontal, TerminalBlock_Phoenix:TerminalBlock_Phoenix_MKDS-1-10-3.81_1x10_P3.81mm_Horizontal
- removed U1 (x2): LTV-817S, Package_DIP:SMDIP-4_W9.53mm

Commit message: modified:   DECON_Ctrl_Panel.kicad_sch
Parts:
- added C1: 330uF/50V, Capacitor_SMD:CP_Elec_10x10.5, F.Cu at (-12.1, 83.1)
- added C10: 104, Capacitor_SMD:C_0805_2012Metric, F.Cu at (-38.9, 69.6)
- added C11: 104, Capacitor_SMD:C_0805_2012Metric, F.Cu at (-38.9, 72.6)
- added C12: 104, Capacitor_SMD:C_0805_2012Metric, F.Cu at (-34.5, 63.5)
- added C13: 104, Capacitor_SMD:C_0805_2012Metric, F.Cu at (-34.5, 66.5)
- added C14: 104, Capacitor_SMD:C_0805_2012Metric, F.Cu at (-34.5, 69.6)
- added C15: 104, Capacitor_SMD:C_0805_2012Metric, F.Cu at (-34.5, 72.6)
- added C16: 104, Capacitor_SMD:C_0805_2012Metric, F.Cu at (-30.0, 63.5)
- added C17: 104, Capacitor_SMD:C_0805_2012Metric, F.Cu at (-30.0, 66.5)
- added C18: 104, Capacitor_SMD:C_0805_2012Metric, F.Cu at (-30.0, 69.6)
- added C19: 104, Capacitor_SMD:C_0805_2012Metric, F.Cu at (-30.0, 72.6)
- added C2: 1nF/2kV, Capacitor_THT:C_Disc_D5.0mm_W2.5mm_P5.00mm, F.Cu at (-12.1, 111.2)
- added C20: 104, Capacitor_SMD:C_0805_2012Metric, F.Cu at (-25.6, 63.5)
- added C21: 104, Capacitor_SMD:C_0805_2012Metric, F.Cu at (-25.6, 66.5)
- added C22: 104, Capacitor_SMD:C_0805_2012Metric, F.Cu at (-25.6, 69.6)
- added C23: 104, Capacitor_SMD:C_0805_2012Metric, F.Cu at (-25.6, 72.6)
- added C3: 1uF/50V, Capacitor_SMD:C_0805_2012Metric, F.Cu at (-11.4, 118.8)
- added C4: 330uF/50V, Capacitor_SMD:CP_Elec_10x10.5, F.Cu at (-12.1, 95.2)
- added C5: 1nF/2kV, Capacitor_THT:C_Disc_D5.0mm_W2.5mm_P5.00mm, F.Cu at (-12.1, 115.2)
- added C6: 10uF/16V, Capacitor_SMD:CP_Elec_4x5.4, F.Cu at (-17.5, 107.2)
- added C7: 22uF/16V, Capacitor_SMD:CP_Elec_4x5.4, F.Cu at (-17.5, 113.0)
- added C8: 104, Capacitor_SMD:C_0805_2012Metric, F.Cu at (-38.9, 63.5)
- added C9: 104, Capacitor_SMD:C_0805_2012Metric, F.Cu at (-38.9, 66.5)
- added D1: LED, LED_SMD:LED_0805_2012Metric, F.Cu at (-24.4, 113.7)
- added D10: 1N4148W, Diode_SMD:D_SOD-123, F.Cu at (-55.9, 66.7)
- added D11: 1N4148W, Diode_SMD:D_SOD-123, F.Cu at (-55.9, 70.0)
- added D12: LED, LED_SMD:LED_0805_2012Metric, F.Cu at (-34.5, 54.4)
- added D13: LED, LED_SMD:LED_0805_2012Metric, F.Cu at (-34.5, 57.5)
- added D14: 1N4148W, Diode_SMD:D_SOD-123, F.Cu at (-55.9, 73.4)
- added D15: 1N4148W, Diode_SMD:D_SOD-123, F.Cu at (-50.1, 56.6)
- added D16: LED, LED_SMD:LED_0805_2012Metric, F.Cu at (-34.5, 60.5)
- added D17: LED, LED_SMD:LED_0805_2012Metric, F.Cu at (-30.0, 51.4)
- added D18: 1N4148W, Diode_SMD:D_SOD-123, F.Cu at (-50.1, 60.0)
- added D19: 1N4148W, Diode_SMD:D_SOD-123, F.Cu at (-50.1, 63.4)
- added D2: LED, LED_SMD:LED_0805_2012Metric, F.Cu at (-38.9, 51.4)
- added D20: LED, LED_SMD:LED_0805_2012Metric, F.Cu at (-30.0, 54.4)
- added D21: LED, LED_SMD:LED_0805_2012Metric, F.Cu at (-30.0, 57.5)
- added D22: 1N4148W, Diode_SMD:D_SOD-123, F.Cu at (-50.1, 66.7)
- added D23: 1N4148W, Diode_SMD:D_SOD-123, F.Cu at (-50.1, 70.0)
- added D24: LED, LED_SMD:LED_0805_2012Metric, F.Cu at (-30.0, 60.5)
- added D25: LED, LED_SMD:LED_0805_2012Metric, F.Cu at (-25.6, 51.4)
- added D26: 1N4148W, Diode_SMD:D_SOD-123, F.Cu at (-50.1, 73.4)
- added D27: 1N4148W, Diode_SMD:D_SOD-123, F.Cu at (-44.3, 56.6)
- added D28: LED, LED_SMD:LED_0805_2012Metric, F.Cu at (-25.6, 54.4)
- added D29: LED, LED_SMD:LED_0805_2012Metric, F.Cu at (-25.6, 57.5)
- added D3: 1N4148W, Diode_SMD:D_SOD-123, F.Cu at (-55.9, 56.6)
- added D30: 1N4148W, Diode_SMD:D_SOD-123, F.Cu at (-44.3, 60.0)
- added D31: 1N4148W, Diode_SMD:D_SOD-123, F.Cu at (-44.3, 63.4)
- added D33: LED, LED_SMD:LED_0805_2012Metric, F.Cu at (-25.6, 60.5)
- added D37: 1N4148W, Diode_SMD:D_SOD-123, F.Cu at (-44.3, 66.7)
- added D4: LED, LED_SMD:LED_0805_2012Metric, F.Cu at (-38.9, 54.4)
- added D5: LED, LED_SMD:LED_0805_2012Metric, F.Cu at (-38.9, 57.5)
- added D6: 1N4148W, Diode_SMD:D_SOD-123, F.Cu at (-55.9, 60.0)
- added D7: 1N4148W, Diode_SMD:D_SOD-123, F.Cu at (-55.9, 63.4)
- added D8: LED, LED_SMD:LED_0805_2012Metric, F.Cu at (-38.9, 60.5)
- added D9: LED, LED_SMD:LED_0805_2012Metric, F.Cu at (-34.5, 51.4)
- added F1: Fuse, Fuse:Fuseholder_Clip-5x20mm_Eaton_1A5601-01_Inline_P20.80x6.76mm_D1.70mm_Horizontal, F.Cu at (-44.3, 108.2)
- added J21: Conn_01x10, Connector_Phoenix_MC:PhoenixContact_MC_1,5_10-G-3.81_1x10_P3.81mm_Horizontal, F.Cu at (-86.3, 80.2)
- added J22: Conn_01x10, Connector_Phoenix_MC:PhoenixContact_MC_1,5_10-G-3.81_1x10_P3.81mm_Horizontal, F.Cu at (-86.3, 92.4)
- added J24: Conn_01x10, Connector_Phoenix_MC:PhoenixContact_MC_1,5_10-G-3.81_1x10_P3.81mm_Horizontal, F.Cu at (-99.4, 65.8)
- added K1: G5NB, Relay_THT:Relay_SPST_Omron_G5NB, F.Cu at (-101.2, -6.25)
- added K10: G5NB, Relay_THT:Relay_SPST_Omron_G5NB, F.Cu at (-79.0, 2.64)
- added K11: G5NB, Relay_THT:Relay_SPST_Omron_G5NB, F.Cu at (-79.0, 11.5)
- added K12: G5NB, Relay_THT:Relay_SPST_Omron_G5NB, F.Cu at (-79.0, 20.4)
- added K13: G5NB, Relay_THT:Relay_SPST_Omron_G5NB, F.Cu at (-79.0, 29.3)
- added K14: G5NB, Relay_THT:Relay_SPST_Omron_G5NB, F.Cu at (-79.0, 38.2)
- added K15: G5NB, Relay_THT:Relay_SPST_Omron_G5NB, F.Cu at (-79.0, 47.1)
- added K17: G5NB, Relay_THT:Relay_SPST_Omron_G5NB, F.Cu at (-79.0, 56.0)
- added K2: G5NB, Relay_THT:Relay_SPST_Omron_G5NB, F.Cu at (-101.2, 2.64)
- added K3: G5NB, Relay_THT:Relay_SPST_Omron_G5NB, F.Cu at (-101.2, 11.5)
- added K4: G5NB, Relay_THT:Relay_SPST_Omron_G5NB, F.Cu at (-101.2, 20.4)
- added K5: G5NB, Relay_THT:Relay_SPST_Omron_G5NB, F.Cu at (-101.2, 29.3)
- added K6: G5NB, Relay_THT:Relay_SPST_Omron_G5NB, F.Cu at (-101.2, 38.2)
- added K7: G5NB, Relay_THT:Relay_SPST_Omron_G5NB, F.Cu at (-101.2, 47.1)
- added K8: G5NB, Relay_THT:Relay_SPST_Omron_G5NB, F.Cu at (-101.2, 56.0)
- added K9: G5NB, Relay_THT:Relay_SPST_Omron_G5NB, F.Cu at (-79.0, -6.25)
- added L1: 4.7uH, Inductor_SMD:L_APV_APH0630, F.Cu at (-41.5, 116.3)
- added Q1: MMBT2222A, Package_TO_SOT_SMD:SOT-23-3, F.Cu at (-38.6, 33.8)
- added Q10: MMBT2222A, Package_TO_SOT_SMD:SOT-23-3, F.Cu at (-28.3, 38.4)
- added Q11: MMBT2222A, Package_TO_SOT_SMD:SOT-23-3, F.Cu at (-28.3, 43.0)
- added Q12: MMBT2222A, Package_TO_SOT_SMD:SOT-23-3, F.Cu at (-28.3, 47.6)
- added Q13: MMBT2222A, Package_TO_SOT_SMD:SOT-23-3, F.Cu at (-23.1, 33.8)
- added Q14: MMBT2222A, Package_TO_SOT_SMD:SOT-23-3, F.Cu at (-23.1, 38.4)
- added Q15: MMBT2222A, Package_TO_SOT_SMD:SOT-23-3, F.Cu at (-23.1, 43.0)
- added Q17: MMBT2222A, Package_TO_SOT_SMD:SOT-23-3, F.Cu at (-23.1, 47.6)
- added Q2: MMBT2222A, Package_TO_SOT_SMD:SOT-23-3, F.Cu at (-38.6, 38.4)
- added Q3: MMBT2222A, Package_TO_SOT_SMD:SOT-23-3, F.Cu at (-38.6, 43.0)
- added Q4: MMBT2222A, Package_TO_SOT_SMD:SOT-23-3, F.Cu at (-38.6, 47.6)
- added Q5: MMBT2222A, Package_TO_SOT_SMD:SOT-23-3, F.Cu at (-33.4, 33.8)
- added Q6: MMBT2222A, Package_TO_SOT_SMD:SOT-23-3, F.Cu at (-33.4, 38.4)
- added Q7: MMBT2222A, Package_TO_SOT_SMD:SOT-23-3, F.Cu at (-33.4, 43.0)
- added Q8: MMBT2222A, Package_TO_SOT_SMD:SOT-23-3, F.Cu at (-33.4, 47.6)
- added Q9: MMBT2222A, Package_TO_SOT_SMD:SOT-23-3, F.Cu at (-28.3, 33.8)
- added R1: R, Resistor_SMD:R_0805_2012Metric, F.Cu at (-24.4, 116.7)
- added R10: 510, Resistor_SMD:R_0805_2012Metric, F.Cu at (-52.2, 32.9)
- added R11: 510, Resistor_SMD:R_0805_2012Metric, F.Cu at (-52.2, 35.8)
- added R12: 1K, Resistor_SMD:R_0805_2012Metric, F.Cu at (-52.2, 38.8)
- added R13: 1K, Resistor_SMD:R_0805_2012Metric, F.Cu at (-52.2, 41.7)
- added R14: 510, Resistor_SMD:R_0805_2012Metric, F.Cu at (-52.2, 44.6)
- added R15: 510, Resistor_SMD:R_0805_2012Metric, F.Cu at (-52.2, 47.6)
- added R16: 1K, Resistor_SMD:R_0805_2012Metric, F.Cu at (-52.2, 50.5)
- added R17: 1K, Resistor_SMD:R_0805_2012Metric, F.Cu at (-52.2, 53.5)
- added R18: 510, Resistor_SMD:R_0805_2012Metric, F.Cu at (-47.8, 32.9)
- added R19: 510, Resistor_SMD:R_0805_2012Metric, F.Cu at (-47.8, 35.8)
- added R2: 1K, Resistor_SMD:R_0805_2012Metric, F.Cu at (-56.6, 32.9)
- added R20: 1K, Resistor_SMD:R_0805_2012Metric, F.Cu at (-47.8, 38.8)
- added R21: 1K, Resistor_SMD:R_0805_2012Metric, F.Cu at (-47.8, 41.7)
- added R22: 510, Resistor_SMD:R_0805_2012Metric, F.Cu at (-47.8, 44.6)
- added R23: 510, Resistor_SMD:R_0805_2012Metric, F.Cu at (-47.8, 47.6)
- added R24: 1K, Resistor_SMD:R_0805_2012Metric, F.Cu at (-47.8, 50.5)
- added R25: 1K, Resistor_SMD:R_0805_2012Metric, F.Cu at (-47.8, 53.5)
- added R26: 510, Resistor_SMD:R_0805_2012Metric, F.Cu at (-43.4, 32.9)
- added R27: 510, Resistor_SMD:R_0805_2012Metric, F.Cu at (-43.4, 35.8)
- added R28: 1K, Resistor_SMD:R_0805_2012Metric, F.Cu at (-43.4, 38.8)
- added R29: 1K, Resistor_SMD:R_0805_2012Metric, F.Cu at (-43.4, 41.7)
- added R3: 510, Resistor_SMD:R_0805_2012Metric, F.Cu at (-56.6, 35.8)
- added R30: 510, Resistor_SMD:R_0805_2012Metric, F.Cu at (-43.4, 44.6)
- added R31: 510, Resistor_SMD:R_0805_2012Metric, F.Cu at (-43.4, 47.6)
- added R33: 1K, Resistor_SMD:R_0805_2012Metric, F.Cu at (-43.4, 50.5)
- added R37: 510, Resistor_SMD:R_0805_2012Metric, F.Cu at (-43.4, 53.5)
- added R4: 1K, Resistor_SMD:R_0805_2012Metric, F.Cu at (-56.6, 38.8)
- added R43: 1K, Resistor_SMD:R_0805_2012Metric, F.Cu at (-87.9, 102.9)
- added R44: 1K, Resistor_SMD:R_0805_2012Metric, F.Cu at (-87.9, 105.9)
- added R47: 1K, Resistor_SMD:R_0805_2012Metric, F.Cu at (-87.9, 108.8)
- added R48: 1K, Resistor_SMD:R_0805_2012Metric, F.Cu at (-87.9, 111.8)
- added R49: 1K, Resistor_SMD:R_0805_2012Metric, F.Cu at (-87.9, 114.7)
- added R5: 1K, Resistor_SMD:R_0805_2012Metric, F.Cu at (-56.6, 41.7)
- added R50: 1K, Resistor_SMD:R_0805_2012Metric, F.Cu at (-87.9, 117.7)
- added R51: 1K, Resistor_SMD:R_0805_2012Metric, F.Cu at (-87.9, 120.6)
- added R52: 1K, Resistor_SMD:R_0805_2012Metric, F.Cu at (-83.5, 102.9)
- added R53: 1K, Resistor_SMD:R_0805_2012Metric, F.Cu at (-83.5, 105.9)
- added R54: 1K, Resistor_SMD:R_0805_2012Metric, F.Cu at (-83.5, 108.8)
- added R6: 510, Resistor_SMD:R_0805_2012Metric, F.Cu at (-56.6, 44.6)
- added R65: 10K, Resistor_SMD:R_0805_2012Metric, F.Cu at (-83.5, 111.8)
- added R66: 10K, Resistor_SMD:R_0805_2012Metric, F.Cu at (-83.5, 114.7)
- added R67: 10K, Resistor_SMD:R_0805_2012Metric, F.Cu at (-83.5, 117.7)
- added R68: 10K, Resistor_SMD:R_0805_2012Metric, F.Cu at (-83.5, 120.6)
- added R69: 10K, Resistor_SMD:R_0805_2012Metric, F.Cu at (-79.1, 102.9)
- added R7: 510, Resistor_SMD:R_0805_2012Metric, F.Cu at (-56.6, 47.6)
- added R70: 10K, Resistor_SMD:R_0805_2012Metric, F.Cu at (-79.1, 105.9)
- added R71: 1K, Resistor_SMD:R_0805_2012Metric, F.Cu at (-79.1, 108.8)
- added R72: 1K, Resistor_SMD:R_0805_2012Metric, F.Cu at (-79.1, 111.8)
- added R73: 1K, Resistor_SMD:R_0805_2012Metric, F.Cu at (-79.1, 114.7)
- added R74: 1K, Resistor_SMD:R_0805_2012Metric, F.Cu at (-79.1, 117.7)
- added R75: 1K, Resistor_SMD:R_0805_2012Metric, F.Cu at (-79.1, 120.6)
- added R76: 1K, Resistor_SMD:R_0805_2012Metric, F.Cu at (-74.6, 102.9)
- added R77: 10K, Resistor_SMD:R_0805_2012Metric, F.Cu at (-74.6, 105.9)
- added R78: 10K, Resistor_SMD:R_0805_2012Metric, F.Cu at (-74.6, 108.8)
- added R79: 10K, Resistor_SMD:R_0805_2012Metric, F.Cu at (-74.6, 111.8)
- added R8: 1K, Resistor_SMD:R_0805_2012Metric, F.Cu at (-56.6, 50.5)
- added R80: 10K, Resistor_SMD:R_0805_2012Metric, F.Cu at (-74.6, 114.7)
- added R81: 10K, Resistor_SMD:R_0805_2012Metric, F.Cu at (-74.6, 117.7)
- added R82: 10K, Resistor_SMD:R_0805_2012Metric, F.Cu at (-74.6, 120.6)
- added R83: 10K, Resistor_SMD:R_0805_2012Metric, F.Cu at (-70.2, 102.9)
- added R84: 10K, Resistor_SMD:R_0805_2012Metric, F.Cu at (-70.2, 105.9)
- added R85: 10K, Resistor_SMD:R_0805_2012Metric, F.Cu at (-70.2, 108.8)
- added R86: 10K, Resistor_SMD:R_0805_2012Metric, F.Cu at (-70.2, 111.8)
- added R87: 10K, Resistor_SMD:R_0805_2012Metric, F.Cu at (-70.2, 114.7)
- added R88: 10K, Resistor_SMD:R_0805_2012Metric, F.Cu at (-70.2, 117.7)
- added R89: 10K, Resistor_SMD:R_0805_2012Metric, F.Cu at (-70.2, 120.6)
- added R9: 1K, Resistor_SMD:R_0805_2012Metric, F.Cu at (-56.6, 53.5)
- added RV1: Varistor, Varistor:RV_Disc_D7mm_W3.4mm_P5mm, F.Cu at (-11.9, 106.0)
- added U1: URB2405YMD-10WR3, Son_KiCad_lib:URB2405YMD-10WR3, F.Cu at (-35.5, 80.6)
- added U10: LTV-817S, Package_DIP:SMDIP-4_W9.53mm, F.Cu at (-52.3, 28.1)
- added U11: LTV-817S, Package_DIP:SMDIP-4_W9.53mm, F.Cu at (-39.2, -5.09)
- added U12: LTV-817S, Package_DIP:SMDIP-4_W9.53mm, F.Cu at (-39.2, 1.54)
- added U13: LTV-817S, Package_DIP:SMDIP-4_W9.53mm, F.Cu at (-39.2, 8.17)
- added U14: LTV-817S, Package_DIP:SMDIP-4_W9.53mm, F.Cu at (-39.2, 14.8)
- added U15: LTV-817S, Package_DIP:SMDIP-4_W9.53mm, F.Cu at (-39.2, 21.4)
- added U16: LTV-817S, Package_DIP:SMDIP-4_W9.53mm, F.Cu at (-39.2, 28.1)
- added U17: LTV-817S, Package_DIP:SMDIP-4_W9.53mm, F.Cu at (-26.1, -5.09)
- added U18: LTV-817S, Package_DIP:SMDIP-4_W9.53mm, F.Cu at (-26.1, 1.54)
- added U19: LTV-817S, Package_DIP:SMDIP-4_W9.53mm, F.Cu at (-26.1, 8.17)
- added U2: 74HC138, Package_SO:SOIC-16_3.9x9.9mm_P1.27mm, F.Cu at (-63.8, 107.3)
- added U20: LTV-817S, Package_DIP:SMDIP-4_W9.53mm, F.Cu at (-26.1, 14.8)
- added U26: LTV-817S, Package_DIP:SMDIP-4_W9.53mm, F.Cu at (-96.6, 80.4)
- added U27: LTV-817S, Package_DIP:SMDIP-4_W9.53mm, F.Cu at (-96.6, 87.0)
- added U3: STM32F401R_B-C_Tx, Package_QFP:LQFP-64_10x10mm_P0.5mm, F.Cu at (-10.3, -1.18)
- added U34: LTV-817S, Package_DIP:SMDIP-4_W9.53mm, F.Cu at (-96.6, 93.7)
- added U35: LTV-817S, Package_DIP:SMDIP-4_W9.53mm, F.Cu at (-96.6, 100.3)
- added U36: LTV-817S, Package_DIP:SMDIP-4_W9.53mm, F.Cu at (-96.6, 106.9)
- added U37: LTV-817S, Package_DIP:SMDIP-4_W9.53mm, F.Cu at (-96.6, 113.5)
- added U38: LTV-817S, Package_DIP:SMDIP-4_W9.53mm, F.Cu at (-96.6, 120.2)
- added U39: LTV-817S, Package_DIP:SMDIP-4_W9.53mm, F.Cu at (-96.6, 126.8)
- added U4: AZ1117-3.3, Package_TO_SOT_SMD:SOT-223-3_TabPin2, F.Cu at (-31.6, 116.4)
- added U5: LTV-817S, Package_DIP:SMDIP-4_W9.53mm, F.Cu at (-52.3, -5.09)
- added U6: LTV-817S, Package_DIP:SMDIP-4_W9.53mm, F.Cu at (-52.3, 1.54)
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Other:
- board size 150 x 90 mm -> 194.1 x 106.1 mm

Commit message: modified:   DECON_Ctrl_Panel.kicad_pcb
Parts:
- added REF**: PhoenixContact_MC_1,5_10-G-3.81_1x10_P3.81mm_Horizontal, Connector_Phoenix_MC:PhoenixContact_MC_1,5_10-G-3.81_1x10_P3.81mm_Horizontal, F.Cu at (74.4, -36.6)

Commit message: modified:   DECON_Ctrl_Panel.kicad_pcb
Parts:
- added REF**: TerminalBlock_Phoenix_MKDS-3-10-5.08_1x10_P5.08mm_Horizontal, TerminalBlock_Phoenix:TerminalBlock_Phoenix_MKDS-3-10-5.08_1x10_P5.08mm_Horizontal, F.Cu at (55.5, 160.5)
- added REF**: Crystal_SMD_Abracon_ABS25-4Pin_8.0x3.8mm, Crystal:Crystal_SMD_Abracon_ABS25-4Pin_8.0x3.8mm, F.Cu at (33.0, 130.0)
- added REF**: TerminalBlock_Phoenix_MKDS-1,5-16-5.08_1x16_P5.08mm_Horizon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, TerminalBlock_Phoenix:TerminalBlock_Phoenix_MKDS-1,5-16-5.08_1x16_P5.08mm_Horizontal, F.Cu at (132.5, 211.5)
- added REF**: SW_SPST_CK_RS282G05A3, Button_Switch_SMD:SW_SPST_CK_RS282G05A3, F.Cu at (21.5, -5.50)
- added REF**: TerminalBlock_Phoenix_MKDS-1,5-5-5.08_1x05_P5.08mm_Horizont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, TerminalBlock_Phoenix:TerminalBlock_Phoenix_MKDS-1,5-5-5.08_1x05_P5.08mm_Horizontal, F.Cu at (129.5, 117.0)
- added REF**: Crystal_SMD_3225-4Pin_3.2x2.5mm, Crystal:Crystal_SMD_3225-4Pin_3.2x2.5mm, F.Cu at (47.5, 129.5)
- added REF**: TerminalBlock_Phoenix_MKDS-3-10-5.08_1x10_P5.08mm_Horizontal, TerminalBlock_Phoenix:TerminalBlock_Phoenix_MKDS-3-10-5.08_1x10_P5.08mm_Horizontal, F.Cu at (107.5, 160.5)

Commit message: modified:   DECON_Ctrl_Panel.kicad_pcb
Parts:
- removed D37: 1N4148W, Diode_SMD:D_SOD-123
- removed J21, J22, J24: Conn_01x10, Connector_Phoenix_MC:PhoenixContact_MC_1,5_10-G-3.81_1x10_P3.81mm_Horizontal
- removed Q17: MMBT2222A, Package_TO_SOT_SMD:SOT-23-3
- removed REF**: PhoenixContact_MC_1,5_10-G-3.81_1x10_P3.81mm_Horizontal, Connector_Phoenix_MC:PhoenixContact_MC_1,5_10-G-3.81_1x10_P3.81mm_Horizontal
- removed REF** (x2): TerminalBlock_Phoenix_MKDS-3-10-5.08_1x10_P5.08mm_Horizontal, TerminalBlock_Phoenix:TerminalBlock_Phoenix_MKDS-3-10-5.08_1x10_P5.08mm_Horizontal
- removed REF**: Crystal_SMD_Abracon_ABS25-4Pin_8.0x3.8mm, Crystal:Crystal_SMD_Abracon_ABS25-4Pin_8.0x3.8mm
- removed REF**: TerminalBlock_Phoenix_MKDS-1,5-16-5.08_1x16_P5.08mm_Horizon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, TerminalBlock_Phoenix:TerminalBlock_Phoenix_MKDS-1,5-16-5.08_1x16_P5.08mm_Horizontal
- removed REF**: SW_SPST_CK_RS282G05A3, Button_Switch_SMD:SW_SPST_CK_RS282G05A3
- removed REF**: TerminalBlock_Phoenix_MKDS-1,5-5-5.08_1x05_P5.08mm_Horizont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, TerminalBlock_Phoenix:TerminalBlock_Phoenix_MKDS-1,5-5-5.08_1x05_P5.08mm_Horizontal
- removed REF**: Crystal_SMD_3225-4Pin_3.2x2.5mm, Crystal:Crystal_SMD_3225-4Pin_3.2x2.5mm
- removed U37, U38, U39: LTV-817S, Package_DIP:SMDIP-4_W9.53mm
- added C24: 104, Capacitor_SMD:C_0805_2012Metric, F.Cu at (162.9, -14.9)
- added C25: 104, Capacitor_SMD:C_0805_2012Metric, F.Cu at (162.9, -11.9)
- added C26: 104, Capacitor_SMD:C_0805_2012Metric, F.Cu at (167.4, -20.9)
- added C27: 104, Capacitor_SMD:C_0805_2012Metric, F.Cu at (167.4, -17.9)
- added C28: 104, Capacitor_SMD:C_0805_2012Metric, F.Cu at (167.4, -14.9)
- added C29: 104, Capacitor_SMD:C_0805_2012Metric, F.Cu at (167.4, -11.9)
- added C30: 104, Capacitor_SMD:C_0805_2012Metric, F.Cu at (171.8, -20.9)
- added C31: 104, Capacitor_SMD:C_0805_2012Metric, F.Cu at (171.8, -17.9)
- added C32: 104, Capacitor_SMD:C_0805_2012Metric, F.Cu at (171.8, -14.9)
- added C33: 104, Capacitor_SMD:C_0805_2012Metric, F.Cu at (171.8, -11.9)
- added C34: 104, Capacitor_SMD:C_0805_2012Metric, F.Cu at (176.3, -20.9)
- added C35: 104, Capacitor_SMD:C_0805_2012Metric, F.Cu at (176.3, -17.9)
- added C36: 104, Capacitor_SMD:C_0805_2012Metric, F.Cu at (176.3, -14.9)
- added C37: 104, Capacitor_SMD:C_0805_2012Metric, F.Cu at (176.3, -11.9)
- added D32: 1N4148W, Diode_SMD:D_SOD-123, F.Cu at (178.8, 12.0)
- added D34: LED, LED_SMD:LED_0805_2012Metric, F.Cu at (176.3, -23.9)
- added J11: Conn_01x06, TerminalBlock_MetzConnect:TerminalBlock_MetzConnect_Type086_RT03406HBLC_1x06_P3.81mm_Horizontal, F.Cu at (64.1, 167.7)
- added J12: Conn_01x06, TerminalBlock_MetzConnect:TerminalBlock_MetzConnect_Type086_RT03406HBLC_1x06_P3.81mm_Horizontal, F.Cu at (64.1, 177.3)
- added J13: Conn_01x02, TerminalBlock_MetzConnect:TerminalBlock_MetzConnect_Type086_RT03402HBLC_1x02_P3.81mm_Horizontal, F.Cu at (53.1, -15.3)
- added J14: Conn_01x06, TerminalBlock_MetzConnect:TerminalBlock_MetzConnect_Type086_RT03406HBLC_1x06_P3.81mm_Horizontal, F.Cu at (20.2, -15.8)
- added J15: Conn_01x06, TerminalBlock_MetzConnect:TerminalBlock_MetzConnect_Type086_RT03406HBLC_1x06_P3.81mm_Horizontal, F.Cu at (20.2, -6.19)
- added J16: Conn_01x06, TerminalBlock_MetzConnect:TerminalBlock_MetzConnect_Type086_RT03406HBLC_1x06_P3.81mm_Horizontal, F.Cu at (20.2, 3.43)
- added J4: GPIO, Connector_PinHeader_2.54mm:PinHeader_1x12_P2.54mm_Vertical, F.Cu at (197.5, 60.2)
- added J5: FLASH, Connector_PinHeader_1.00mm:PinHeader_1x08_P1.00mm_Vertical, F.Cu at (198.4, 68.6)
- added J7: Conn_01x06, TerminalBlock_MetzConnect:TerminalBlock_MetzConnect_Type086_RT03406HBLC_1x06_P3.81mm_Horizontal, F.Cu at (64.1, 148.4)
- added J8: Conn_01x06, TerminalBlock_MetzConnect:TerminalBlock_MetzConnect_Type086_RT03406HBLC_1x06_P3.81mm_Horizontal, F.Cu at (64.1, 158.1)
- added K16: G5NB, Relay_THT:Relay_SPST_Omron_G5NB, F.Cu at (140.5, -24.2)
- added Q16: MMBT2222A, Package_TO_SOT_SMD:SOT-23-3, F.Cu at (178.7, -36.8)
- added R100: 10K, Resistor_SMD:R_0805_2012Metric, F.Cu at (220.7, 200.0)
- added R101: 1K, Resistor_SMD:R_0805_2012Metric, F.Cu at (220.7, 203.0)
- added R102: 10K, Resistor_SMD:R_0805_2012Metric, F.Cu at (220.7, 205.9)
- added R103: 1K, Resistor_SMD:R_0805_2012Metric, F.Cu at (220.7, 208.9)
- added R104: 1K, Resistor_SMD:R_0805_2012Metric, F.Cu at (150.3, 211.6)
- added R105: 1K, Resistor_SMD:R_0805_2012Metric, F.Cu at (154.7, 188.0)
- added R106: 10K, Resistor_SMD:R_0805_2012Metric, F.Cu at (225.1, 191.2)
- added R107: 1K, Resistor_SMD:R_0805_2012Metric, F.Cu at (154.7, 193.9)
- added R108: 1K, Resistor_SMD:R_0805_2012Metric, F.Cu at (154.7, 196.8)
- added R109: 1K, Resistor_SMD:R_0805_2012Metric, F.Cu at (225.1, 200.0)
- added R110: 1K, Resistor_SMD:R_0805_2012Metric, F.Cu at (154.7, 202.7)
- added R111: 1K, Resistor_SMD:R_0805_2012Metric, F.Cu at (154.7, 205.7)
- added R112: 10K, Resistor_SMD:R_0805_2012Metric, F.Cu at (225.1, 208.9)
- added R113: 1K, Resistor_SMD:R_0805_2012Metric, F.Cu at (225.1, 211.8)
- added R114: 1K, Resistor_SMD:R_0805_2012Metric, F.Cu at (159.1, 188.0)
- added R115: 1K, Resistor_SMD:R_0805_2012Metric, F.Cu at (159.1, 190.9)
- added R116: 10K, Resistor_SMD:R_0805_2012Metric, F.Cu at (229.5, 194.1)
- added R117: 1K, Resistor_SMD:R_0805_2012Metric, F.Cu at (229.5, 197.1)
- added R118: 1K, Resistor_SMD:R_0805_2012Metric, F.Cu at (159.1, 199.8)
- added R119: 1K, Resistor_SMD:R_0805_2012Metric, F.Cu at (159.1, 202.7)
- added R120: 10K, Resistor_SMD:R_0805_2012Metric, F.Cu at (229.5, 205.9)
- added R121: 1K, Resistor_SMD:R_0805_2012Metric, F.Cu at (159.1, 208.6)
- added R122: 1K, Resistor_SMD:R_0805_2012Metric, F.Cu at (159.1, 211.6)
- added R123: 1K, Resistor_SMD:R_0805_2012Metric, F.Cu at (233.9, 188.2)
- added R124: 1K, Resistor_SMD:R_0805_2012Metric, F.Cu at (163.6, 190.9)
- added R125: 1K, Resistor_SMD:R_0805_2012Metric, F.Cu at (163.6, 193.9)
- added R126: 1K, Resistor_SMD:R_0805_2012Metric, F.Cu at (163.6, 196.8)
- added R127: 1K, Resistor_SMD:R_0805_2012Metric, F.Cu at (163.6, 199.8)
- added R128: 1K, Resistor_SMD:R_0805_2012Metric, F.Cu at (163.6, 202.7)
- added R129: 1K, Resistor_SMD:R_0805_2012Metric, F.Cu at (163.6, 205.7)
- added R32: 1K, Resistor_SMD:R_0805_2012Metric, F.Cu at (144.4, 7.62)
- added R34: 10K, Resistor_SMD:R_0805_2012Metric, F.Cu at (144.4, 13.5)
- added R35: 10K, Resistor_SMD:R_0805_2012Metric, F.Cu at (144.4, 16.5)
- added R36: 10K, Resistor_SMD:R_0805_2012Metric, F.Cu at (144.4, 19.4)
- added R38: 10K, Resistor_SMD:R_0805_2012Metric, F.Cu at (144.4, 25.3)
- added R39: 1K, Resistor_SMD:R_0805_2012Metric, F.Cu at (144.4, 28.3)
- added R40: 10K, Resistor_SMD:R_0805_2012Metric, F.Cu at (144.4, 31.2)
- added R41: 1K, Resistor_SMD:R_0805_2012Metric, F.Cu at (144.4, 34.2)
- added R42: 470, Resistor_SMD:R_0805_2012Metric, F.Cu at (148.8, 1.72)
- added R45: 1K, Resistor_SMD:R_0805_2012Metric, F.Cu at (148.8, 10.6)
- added R46: 1K, Resistor_SMD:R_0805_2012Metric, F.Cu at (148.8, 13.5)
- added R55: 10K, Resistor_SMD:R_0805_2012Metric, F.Cu at (153.3, 4.67)
- added R56: 1K, Resistor_SMD:R_0805_2012Metric, F.Cu at (153.3, 7.62)
- added R57: 470, Resistor_SMD:R_0805_2012Metric, F.Cu at (153.3, 10.6)
- added R58: 470, Resistor_SMD:R_0805_2012Metric, F.Cu at (153.3, 13.5)
- added R59: 470, Resistor_SMD:R_0805_2012Metric, F.Cu at (153.3, 16.5)
- added R60: 1K, Resistor_SMD:R_0805_2012Metric, F.Cu at (153.3, 19.4)
- added R61: 1K, Resistor_SMD:R_0805_2012Metric, F.Cu at (153.3, 22.4)
- added R62: 1K, Resistor_SMD:R_0805_2012Metric, F.Cu at (153.3, 25.3)
- added R63: 10K, Resistor_SMD:R_0805_2012Metric, F.Cu at (153.3, 28.3)
- added R64: 10K, Resistor_SMD:R_0805_2012Metric, F.Cu at (153.3, 31.2)
- added R90: 10K, Resistor_SMD:R_0805_2012Metric, F.Cu at (176.9, 109.9)
- added R91: 10K, Resistor_SMD:R_0805_2012Metric, F.Cu at (176.9, 112.9)
- added R92: 10K, Resistor_SMD:R_0805_2012Metric, F.Cu at (176.9, 115.8)
- added R93: 10K, Resistor_SMD:R_0805_2012Metric, F.Cu at (176.9, 118.8)
- added R94: 10K, Resistor_SMD:R_0805_2012Metric, F.Cu at (176.9, 121.7)
- added R95: 10K, Resistor_SMD:R_0805_2012Metric, F.Cu at (176.9, 124.7)
- added R96: 10K, Resistor_SMD:R_0805_2012Metric, F.Cu at (181.3, 101.1)
- added R97: 10K, Resistor_SMD:R_0805_2012Metric, F.Cu at (181.3, 104.0)
- added R98: 10K, Resistor_SMD:R_0805_2012Metric, F.Cu at (220.7, 194.1)
- added R99: 1K, Resistor_SMD:R_0805_2012Metric, F.Cu at (220.7, 197.1)
- added SW1: SW_Push, Button_Switch_SMD:SW_SPST_CK_RS282G05A3, F.Cu at (217.3, 120.8)
- added SW2: SW_Push, Button_Switch_SMD:SW_SPST_CK_RS282G05A3, F.Cu at (217.3, 126.0)
- added U21: 74HC138, Package_SO:SOIC-16_3.9x9.9mm_P1.27mm, F.Cu at (178.9, 132.0)
- added U22: LTV-817S, Package_DIP:SMDIP-4_W9.53mm, F.Cu at (181.3, 196.7)
- added U23: LTV-817S, Package_DIP:SMDIP-4_W9.53mm, F.Cu at (181.3, 203.3)
- added U24: LTV-817S, Package_DIP:SMDIP-4_W9.53mm, F.Cu at (111.0, 209.7)
- added U25: LTV-817S, Package_DIP:SMDIP-4_W9.53mm, F.Cu at (111.0, 216.3)
- added U28: LTV-817S, Package_DIP:SMDIP-4_W9.53mm, F.Cu at (194.4, 196.7)
- added U29: LTV-817S, Package_DIP:SMDIP-4_W9.53mm, F.Cu at (124.1, 203.1)
- added U30: LTV-817S, Package_DIP:SMDIP-4_W9.53mm, F.Cu at (194.4, 209.9)
- added U31: LTV-817S, Package_DIP:SMDIP-4_W9.53mm, F.Cu at (124.1, 216.3)
- added U32: LTV-817S, Package_DIP:SMDIP-4_W9.53mm, F.Cu at (124.1, 223.0)
- added U33: LTV-817S, Package_DIP:SMDIP-4_W9.53mm, F.Cu at (207.5, 190.0)
- added Y1: Crystal, Crystal:Crystal_SMD_3215-2Pin_3.2x1.5mm, F.Cu at (230.6, 102.0)
- added Y2: Crystal_GND24, Crystal:Crystal_SMD_3225-4Pin_3.2x2.5mm, F.Cu at (230.7, 98.1)
- C1: value 330uF/50V -> 1nF/2kV; footprint Capacitor_SMD:CP_Elec_10x10.5 -> Capacitor_THT:C_Disc_D5.0mm_W2.5mm_P5.00mm
- C14: value 104 -> 1nF/2kV; footprint Capacitor_SMD:C_0805_2012Metric -> Capacitor_THT:C_Disc_D5.0mm_W2.5mm_P5.00mm
- C15, C16, C19, C20: value 104 -> 20pF
- C2: value 1nF/2kV -> 330uF/50V; footprint Capacitor_THT:C_Disc_D5.0mm_W2.5mm_P5.00mm -> Capacitor_SMD:CP_Elec_10x10.5
- C21: value 104 -> 2.2uF
- C5: value 1nF/2kV -> 10uF/16V; footprint Capacitor_THT:C_Disc_D5.0mm_W2.5mm_P5.00mm -> Capacitor_SMD:CP_Elec_4x5.4
- C6: value 10uF/16V -> 22uF/16V
- C7: value 22uF/16V -> 104; footprint Capacitor_SMD:CP_Elec_4x5.4 -> Capacitor_SMD:C_0805_2012Metric
- D14, D18, D19, D26, D30, D6, D7: value 1N4148W -> LED; footprint Diode_SMD:D_SOD-123 -> LED_SMD:LED_0805_2012Metric
- D16, D17, D21, D28, D4, D5, D9: value LED -> 1N4148W; footprint LED_SMD:LED_0805_2012Metric -> Diode_SMD:D_SOD-123
- R1: value R -> 1K
- R10, R18, R19, R23, R6: value 510 -> 10K
- R11, R15, R22, R26, R3, R30, R31, R37, R7: value 510 -> 1K
- R12, R13, R28, R29, R43, R44, R71, R72: value 1K -> 470
- R14, R27: value 510 -> 470
- R2, R20, R21, R25, R33, R4, R48, R49, R5, R50, R51, R53, R75, R76, R8: value 1K -> 10K
- R67, R69, R78, R80, R83, R84: value 10K -> 1K
- R70, R81, R82: value 10K -> 470
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Connections:
- C1 pad 1: Net-(C1-Pad1) -> Net-(U2-+VIN)
- C1 pad 2: GND_VBATT -> 5V
- C10 pad 1: RELAY_5 -> GND_MCU
- C10 pad 2: GND_VBAT -> 3.3V
- C11 pad 1: RELAY_8 -> GND_MCU
- C11 pad 2: GND_VBAT -> 3.3V
- C12 pad 1: RELAY_9 -> GND_MCU
- C12 pad 2: GND_VBAT -> 3.3V
- C13 pad 1: RELAY_12 -> GND_MCU
- C13 pad 2: GND_VBAT -> 3.3V
- C14 pad 1: RELAY_13 -> GND_VBATT
- C14 pad 2: GND_VBAT -> GND_MCU
- C15 pad 1: RELAY_2 -> OSC32_IN
- C15 pad 2: GND_VBAT -> GND_MCU
- C16 pad 1: RELAY_3 -> GND_MCU
- C16 pad 2: GND_VBAT -> OSC_IN
- C17 pad 1: RELAY_0 -> MCU_EXTI
- C17 pad 2: GND_VBAT -> GND_MCU
- C18 pad 1: RELAY_6 -> NRST
- C18 pad 2: GND_VBAT -> GND_MCU
- C19 pad 1: RELAY_7 -> GND_MCU
- C19 pad 2: GND_VBAT -> OSC32_OUT
- C2 pad 1: Net-(U1-+VIN) -> Net-(C2-Pad1)
- C2 pad 2: 5V -> GND_VBATT
- C20 pad 1: RELAY_10 -> GND_MCU
- C20 pad 2: GND_VBAT -> OSC_OUT
- C21 pad 1: RELAY_11 -> VCAP1
- C21 pad 2: GND_VBAT -> GND_MCU
- C22 pad 1: RELAY_14 -> RELAY_12
- C23 pad 1: RELAY_15 -> RELAY_0
- C3 pad 1: Net-(C1-Pad1) -> Net-(C2-Pad1)
- C4 pad 1: Net-(U1-+VIN) -> Net-(U2-+VIN)
- C5 pad 1: GND_VBATT -> 5V
- C6 pad 1: 5V -> 3.3V
- C7 pad 1: 3.3v -> GND_MCU
- C7 pad 2: GND_MCU -> 3.3V
- C8 pad 1: RELAY_1 -> GND_MCU
- C8 pad 2: GND_VBAT -> 3.3V
- C9 pad 1: RELAY_4 -> GND_MCU
- C9 pad 2: GND_VBAT -> 3.3V
- D10 pad 1: 3.3V -> V_VALVE
- D11 pad 1: 3.3V -> V_VALVE
- D12 pad 1: MCU_RL12 -> MCU_RL13
- D13 pad 1: MCU_RL13 -> MCU_RL1
- D14 pad 1: 3.3V -> MCU_RL7
- D15 pad 1: 3.3V -> V_VALVE
- D16 pad 1: MCU_RL2 -> V_VALVE
- D17 pad 1: MCU_RL3 -> V_VALVE
- D18 pad 1: 3.3V -> MCU_RL14
- D19 pad 1: 3.3V -> MCU_RL2
- D2 pad 1: MCU_RL1 -> PC13
- D20 pad 1: MCU_RL6 -> MCU_RL8
- D21 pad 1: MCU_RL7 -> V_VALVE
- D22 pad 1: 3.3V -> V_VALVE
- D23 pad 1: 3.3V -> V_VALVE
- D24 pad 1: MCU_RL10 -> MCU_RL15
- D25 pad 1: MCU_RL11 -> MCU_RL3
- D26 pad 1: 3.3V -> MCU_RL9
- D27 pad 1: 3.3V -> V_VALVE
- D28 pad 1: MCU_RL14 -> V_VALVE
- D29 pad 1: MCU_RL15 -> MCU_RL4
- D3 pad 1: 3.3V -> V_VALVE
- D30 pad 1: 3.3V -> MCU_RL10
- D31 pad 1: 3.3V -> V_VALVE
- D33 pad 1: MCU_RL0 -> MCU_RL5
- D4 pad 1: MCU_RL4 -> V_VALVE
- D5 pad 1: MCU_RL5 -> V_VALVE
- D6 pad 1: 3.3V -> MCU_RL12
- D7 pad 1: 3.3V -> MCU_RL0
- D8 pad 1: MCU_RL8 -> MCU_RL6
- D9 pad 1: MCU_RL9 -> V_VALVE
- F1 pad 1: VBATT -> VBAT
- F1 pad 2: Net-(C1-Pad1) -> Net-(C2-Pad1)
- K1 pad 13: RELAY_1 -> RELAY_12
- K1 pad 14: 3.3V -> V_VALVE
- K1 pad A1: 3.3V -> V_VALVE
- K1 pad A2: Net-(D3-A) -> Net-(K1-PadA2)
- K10 pad 13: RELAY_6 -> RELAY_15
- K10 pad 14: 3.3V -> V_VALVE
- K10 pad A1: 3.3V -> V_VALVE
- K10 pad A2: Net-(D22-A) -> Net-(K10-PadA2)
- K11 pad 13: RELAY_7 -> RELAY_3
- K11 pad 14: 3.3V -> V_VALVE
- K11 pad A1: 3.3V -> V_VALVE
- K11 pad A2: Net-(D23-A) -> Net-(K11-PadA2)
- K12 pad 13: RELAY_10 -> RELAY_9
- K12 pad 14: 3.3V -> V_VALVE
- K12 pad A1: 3.3V -> V_VALVE
- K12 pad A2: Net-(D26-A) -> Net-(K12-PadA2)
- K13 pad 13: RELAY_11 -> RELAY_4
- K13 pad 14: 3.3V -> V_VALVE
- K13 pad A1: 3.3V -> V_VALVE
- K13 pad A2: Net-(D27-A) -> Net-(K13-PadA2)
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Other:
- board outline removed

Commit message: modified:   DECON_Ctrl_Panel.kicad_pcb
Parts:
- removed the R12 at (135.6, 19.4)
- removed the R13 at (135.6, 22.4)
- removed the R14 at (135.6, 25.3)
- removed the R27 at (140.0, 28.3)
- removed the R28 at (140.0, 31.2)
- removed the R29 at (140.0, 34.2)
- removed the R42 at (148.8, 1.72)
- removed the R43 at (148.8, 4.67)
- removed the R44 at (148.8, 7.62)
- removed the R57 at (153.3, 10.6)
- removed the R58 at (153.3, 13.5)
- removed the R59 at (153.3, 16.5)
- removed the R70 at (157.7, 13.5)
- removed the R71 at (157.7, 16.5)
- removed the R81 at (162.1, 10.6)
- removed R82: 470, Resistor_SMD:R_0805_2012Metric
- added J10: Conn_01x04, TerminalBlock_MetzConnect:TerminalBlock_MetzConnect_Type086_RT03404HBLC_1x04_P3.81mm_Horizontal, F.Cu at (193.2, 55.5)
- added J13: Conn_01x04, TerminalBlock_MetzConnect:TerminalBlock_MetzConnect_Type086_RT03404HBLC_1x04_P3.81mm_Horizontal, F.Cu at (127.9, 56.0)
- added J18: Conn_01x04, Connector_PinHeader_2.54mm:PinHeader_1x04_P2.54mm_Vertical, F.Cu at (261.3, 168.4)
- added J7: Conn_01x05, TerminalBlock_MetzConnect:TerminalBlock_MetzConnect_Type086_RT03405HBLC_1x05_P3.81mm_Horizontal, F.Cu at (189.4, 152.8)
- C22: renamed from C23; moved to B.Cu
- D10: moved to B.Cu
- D11: renamed from D16; moved to B.Cu
- D12: renamed from D22; moved to B.Cu
- D13: renamed from D27; moved to B.Cu
- D14: renamed from D31; moved to B.Cu
- D21: renamed from D5; moved to B.Cu
- D22: renamed from D11; moved to B.Cu
- D23: renamed from D17; moved to B.Cu
- D24: renamed from D23; moved to B.Cu
- D25: renamed from D28; moved to B.Cu
- D26: renamed from D32; moved to B.Cu
- D31: renamed from D3; moved to B.Cu
- D32: renamed from D9; moved to B.Cu
- D33: renamed from D15; moved to B.Cu
- D34: renamed from D21; moved to B.Cu
- D9: renamed from D4; moved to B.Cu
- J5: footprint Connector_PinHeader_1.00mm:PinHeader_1x08_P1.00mm_Vertical -> Connector_PinHeader_2.54mm:PinHeader_1x08_P2.54mm_Vertical
- moved Q13 304.8 mm to (181.5, 253.6), turned to 180 degrees
- moved Q5 304.5 mm to (166.1, 253.6), turned to 180 degrees
- moved Q9 304.3 mm to (171.2, 253.6), turned to 180 degrees
- moved Q11 295.3 mm to (166.1, 249.0), turned to 180 degrees
- moved Q8 295.1 mm to (176.4, 249.0), turned to 180 degrees
- moved Q16 295.0 mm to (171.2, 249.0), turned to 180 degrees
- moved Q7 286.4 mm to (181.5, 244.4), turned to 180 degrees
- moved Q6 286.1 mm to (166.1, 244.4), turned to 180 degrees
- moved Q15 285.9 mm to (176.4, 244.4), turned to 180 degrees
- moved Q4 285.8 mm to (171.2, 244.4), turned to 180 degrees
- moved Q14 277.1 mm to (181.5, 239.7), turned to 180 degrees
- moved Q12 276.8 mm to (166.1, 239.7), turned to 180 degrees
- moved Q3 276.6 mm to (176.4, 239.7), turned to 180 degrees
- moved Q10 276.5 mm to (171.2, 239.7), turned to 180 degrees
- moved D27 269.7 mm to (181.9, 236.0), turned to 180 degrees
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- renumbered C2 to C1, C19 to C10, C6 to C11, C7 to C12, C16 to C13, C20 to C14, C8 to C15, C9 to C16, C10 to C17, C11 to C18, C12 to C19, C17 to C2, C13 to C20, C26 to C23, C29 to C24, C32 to C25, C34 to C26, C36 to C27, C24 to C28, C27 to C29, C33 to C31, C35 to C32, C37 to C33, C22 to C34, C25 to C35, C28 to C36, C31 to C37, C18 to C5, C1 to C6, C14 to C7, C5 to C8, C15 to C9, D2 to D1, D8 to D15, D14 to D16, D20 to D17, D26 to D18, D30 to D19, D1 to D2, D34 to D20, D6 to D27, D12 to D28, D18 to D29, D7 to D3, D24 to D30, D13 to D4, D19 to D5, D25 to D6, D29 to D7, D33 to D8, J13 to J1, J4 to J2, J14 to J3, J15 to J4, J16 to J6, J7 to J8, J8 to J9, K2 to K1, K12 to K10, K14 to K11, K17 to K12, K1 to K13, K4 to K14, K7 to K15, K10 to K16, K15 to K17, K5 to K2, K8 to K3, K11 to K4, K13 to K5, K16 to K6, K3 to K7, K6 to K8, Q2 to Q1, Q12 to Q10, Q14 to Q11, Q16 to Q12, Q1 to Q13, Q4 to Q14, Q7 to Q15, Q10 to Q16, Q5 to Q2, Q8 to Q3, Q11 to Q4, Q13 to Q5, Q15 to Q6, Q3 to Q7, Q6 to Q8, R3 to R1, R66 to R10, R91 to R100, R92 to R101, R93 to R102, R94 to R103, R95 to R104, R96 to R105, R105 to R106, R108 to R107, R111 to R108, R115 to R109, R77 to R11, R119 to R110, R122 to R111, R125 to R112, R127 to R113, R129 to R114, R97 to R115, R99 to R116, R101 to R117, R103 to R118, R109 to R119, R9 to R12, R113 to R120, R117 to R121, R123 to R122, R98 to R123, R100 to R124, R102 to R125, R106 to R126, R112 to R127, R116 to R128, R120 to R129, R24 to R13, R39 to R14, R54 to R15, R67 to R16, R78 to R17, R16 to R18, R31 to R19, R4 to R2, R46 to R20, R61 to R21, R73 to R22, R83 to R23, R19 to R24, R34 to R25, R49 to R26, R64 to R27, R75 to R28, R85 to R29, R5 to R3, R10 to R36, R25 to R37, R40 to R38, R55 to R39, R1 to R4, R68 to R40, R79 to R41, R11 to R42, R26 to R43, R41 to R44, R56 to R45, R69 to R46, R80 to R47, R17 to R48, R32 to R49, R2 to R5, R47 to R50, R62 to R51, R74 to R52, R84 to R53, R20 to R54, R35 to R55, R50 to R56, R65 to R57, R76 to R58, R86 to R59, R8 to R6, R6 to R66, R21 to R67, R36 to R68, R51 to R69, R23 to R7, R7 to R70, R22 to R71, R37 to R72, R52 to R73, R15 to R74, R30 to R75, R45 to R76, R60 to R77, R18 to R78, R33 to R79, R38 to R8, R48 to R80, R63 to R81, R72 to R86, R53 to R9, R104 to R90, R107 to R91, R110 to R92, R114 to R93, R118 to R94, R121 to R95, R124 to R96, R126 to R97, R128 to R98, R90 to R99, U2 to U1, U6 to U10, U9 to U11, U15 to U13, U17 to U14, U19 to U15, U4 to U16, U7 to U17, U10 to U18, U13 to U19, U1 to U2, U21 to U20, U24 to U21, U25 to U22, U27 to U23, U29 to U24, U31 to U25, U32 to U26, U34 to U27, U35 to U28, U36 to U29, U20 to U30, U22 to U31, U23 to U32, U26 to U33, U28 to U34, U30 to U35, U33 to U36, U5 to U4, U8 to U5, U11 to U6, U14 to U7, U16 to U8, U18 to U9
Connections:
- D11 pad 2: Net-(D16-A) (its old number) -> Net-(D11-A)
- D12 pad 2: Net-(D22-A) -> Net-(D12-A)
- D13 pad 2: Net-(D27-A) (its old number) -> Net-(D13-A)
- D21 pad 2: Net-(D5-A) (its old number) -> Net-(D21-A)
- D22 pad 2: Net-(D11-A) -> Net-(D22-A)
- D24 pad 2: Net-(D23-A) (its old number) -> Net-(D24-A)
- D25 pad 2: Net-(D28-A) (its old number) -> Net-(D25-A)
- D26 pad 1: VBAT -> V_VALVE
- D26 pad 2: Net-(D32-A) -> Net-(D26-A)
- D31 pad 2: Net-(D3-A) (its old number) -> Net-(D31-A)
- D32 pad 2: Net-(D9-A) -> Net-(D32-A)
- D33 pad 2: Net-(D15-A) (its old number) -> Net-(D33-A)
- D34 pad 2: Net-(D21-A) -> Net-(D34-A)
- D9 pad 2: Net-(D4-A) (its old number) -> Net-(D9-A)
- J11 pad 1: BUTTON_0 -> VBAT
- J11 pad 2: BUTTON_1 -> GND_VBAT
- J11 pad 3: BUTTON_2 -> BUTTON_EN
- J11 pad 4: BUTTON_3 -> BUTTON_0
- J11 pad 5: LED_POWER -> BUTTON_1
- J11 pad 6: LED_0 -> BUTTON_2
- J12 pad 1: LED_1 -> BUTTON_3
- J12 pad 2: LED_2 -> LED_POWER
- J12 pad 3: LED_3 -> LED_0
- J12 pad 4: LED_4 -> LED_1
- J12 pad 5: LED_5 -> LED_2
- J12 pad 6: LED_6 -> LED_3
- J3 pad 1: GND_VBAT -> VBAT
- J3 pad 2: RELAY_0 -> GND_VBAT
- J3 pad 3: RELAY_1 -> RELAY_0
- J3 pad 4: RELAY_2 -> RELAY_1
- J3 pad 5: RELAY_3 -> RELAY_2
- J3 pad 6: RELAY_4 -> RELAY_3
- J4 pad 1: RELAY_5 -> RELAY_4
- J4 pad 2: RELAY_6 -> RELAY_5
- J4 pad 3: RELAY_7 -> RELAY_6
- J4 pad 4: RELAY_8 -> RELAY_7
- J4 pad 5: RELAY_9 -> RELAY_8
- J4 pad 6: RELAY_10 -> RELAY_9
- J6 pad 1: RELAY_11 -> RELAY_10
- J6 pad 2: RELAY_12 -> RELAY_11
- J6 pad 3: RELAY_13 -> RELAY_12
- J6 pad 4: RELAY_14 -> RELAY_13
- J6 pad 5: RELAY_15 -> RELAY_14
- J6 pad 6: GND_VBAT -> RELAY_15
- K1 pad 13: RELAY_0 -> V_VALVE
- K1 pad 14: V_VALVE -> RELAY_0
- K1 pad A1: V_VALVE -> Net-(D9-A)
- K1 pad A2: Net-(K2-PadA2) -> V_VALVE
- K10 pad 13: RELAY_9 -> V_VALVE
- K10 pad 14: V_VALVE -> RELAY_9
- K10 pad A1: V_VALVE -> Net-(D24-A)
- K10 pad A2: Net-(K12-PadA2) -> V_VALVE
- K11 pad 13: RELAY_10 -> V_VALVE
- K11 pad 14: V_VALVE -> RELAY_10
- K11 pad A1: V_VALVE -> Net-(D25-A)
- K11 pad A2: Net-(K14-PadA2) -> V_VALVE
- K12 pad 13: RELAY_11 -> V_VALVE
- K12 pad 14: VBAT -> RELAY_11
- K12 pad A1: VBAT -> Net-(D26-A)
- K12 pad A2: Net-(K17-PadA2) (its old number) -> V_VALVE
- K13 pad 13: RELAY_12 -> V_VALVE
- K13 pad 14: V_VALVE -> RELAY_12
- K13 pad A1: V_VALVE -> Net-(D31-A)
- K13 pad A2: Net-(K1-PadA2) -> V_VALVE
- K14 pad 13: RELAY_13 -> V_VALVE
- K14 pad 14: V_VALVE -> RELAY_13
- K14 pad A1: V_VALVE -> Net-(D32-A)
- K14 pad A2: Net-(K4-PadA2) -> V_VALVE
- K15 pad 13: RELAY_14 -> V_VALVE
- K15 pad 14: V_VALVE -> RELAY_14
- K15 pad A1: V_VALVE -> Net-(D33-A)
- K15 pad A2: Net-(K7-PadA2) -> V_VALVE
- K16 pad 13: RELAY_15 -> V_VALVE
- K16 pad 14: V_VALVE -> RELAY_15
- K16 pad A1: V_VALVE -> Net-(D34-A)
- K16 pad A2: Net-(K10-PadA2) -> V_VALVE
- K2 pad 13: RELAY_1 -> V_VALVE
- K2 pad 14: V_VALVE -> RELAY_1
- K2 pad A1: V_VALVE -> Net-(D10-A)
- K2 pad A2: Net-(K5-PadA2) -> V_VALVE
- K3 pad 13: RELAY_2 -> V_VALVE
- K3 pad 14: V_VALVE -> RELAY_2
- K3 pad A1: V_VALVE -> Net-(D11-A)
- K3 pad A2: Net-(K8-PadA2) -> V_VALVE
- K4 pad 13: RELAY_3 -> V_VALVE
- K4 pad 14: V_VALVE -> RELAY_3
- K4 pad A1: V_VALVE -> Net-(D12-A)
- K4 pad A2: Net-(K11-PadA2) -> V_VALVE
- K5 pad 13: RELAY_4 -> V_VALVE
- K5 pad 14: V_VALVE -> RELAY_4
- K5 pad A1: V_VALVE -> Net-(D13-A)
- K5 pad A2: Net-(K13-PadA2) -> V_VALVE
- K6 pad 13: RELAY_5 -> V_VALVE
- K6 pad 14: V_VALVE -> RELAY_5
- K6 pad A1: V_VALVE -> unconnected-(K6-PadA1)
- K6 pad A2: Net-(K16-PadA2) -> V_VALVE
- K7 pad 13: RELAY_6 -> V_VALVE
- K7 pad 14: V_VALVE -> RELAY_6
- K7 pad A1: V_VALVE -> Net-(D21-A)
- K7 pad A2: Net-(K3-PadA2) -> V_VALVE
- K8 pad 13: RELAY_7 -> V_VALVE
- K8 pad 14: V_VALVE -> RELAY_7
- K8 pad A1: V_VALVE -> Net-(D22-A)
- K8 pad A2: Net-(K6-PadA2) -> V_VALVE
- K9 pad 13: RELAY_8 -> V_VALVE
- K9 pad 14: V_VALVE -> RELAY_8
- K9 pad A1: V_VALVE -> unconnected-(K9-PadA1)
- K9 pad A2: Net-(K9-PadA2) -> V_VALVE
- Q1 pad 3: Net-(D4-A) (its old number) -> Net-(D9-A)
- Q10 pad 3: Net-(D23-A) (its old number) -> Net-(D24-A)
- Q11 pad 3: Net-(D28-A) (its old number) -> Net-(D25-A)
- Q12 pad 3: Net-(D32-A) -> Net-(D26-A)
- Q13 pad 3: Net-(D3-A) (its old number) -> Net-(D31-A)
- Q14 pad 3: Net-(D9-A) -> Net-(D32-A)
- Q15 pad 3: Net-(D15-A) (its old number) -> Net-(D33-A)
- Q16 pad 3: Net-(D21-A) -> Net-(D34-A)
- Q3 pad 3: Net-(D16-A) (its old number) -> Net-(D11-A)
- Q4 pad 3: Net-(D22-A) -> Net-(D12-A)
- Q5 pad 3: Net-(D27-A) (its old number) -> Net-(D13-A)
- Q7 pad 3: Net-(D5-A) (its old number) -> Net-(D21-A)
- Q8 pad 3: Net-(D11-A) -> Net-(D22-A)
- U15 pad 4: VBAT -> V_VALVE
Routing:
- net V_VALVE: track 0.00 -> 140.4 mm
- net Net-(R12-Pad2): track 0.00 -> 10.2 mm
- net Net-(D3-A): track 0.00 -> 7.35 mm
- net MCU_RL0: track 0.00 -> 5.50 mm
- net Net-(Q1-B): track 0.00 -> 4.61 mm
- net Net-(R18-Pad1): track 0.00 -> 3.97 mm
- net Net-(D9-A): track 0.00 -> 3.68 mm
Other:
- board outline added: 174 x 106 mm
