File: DECON_Ctrl_Panel.kicad_pcb (KiCad board)
At the start: 2 copper layers, 174 x 106 mm, 274 parts, among them J1 Conn_01x02, J10 Conn_01x04, J11 Conn_01x06, J12 Conn_01x06, J13 Conn_01x04, J18 Conn_01x04, J2 GPIO, J3 Conn_01x06, J4 Conn_01x06, J5 FLASH, J6 Conn_01x06, J7 Conn_01x05, J8 Conn_01x06, J9 Conn_01x06, K1 G5NB, K10 G5NB, K11 G5NB, K12 G5NB, K13 G5NB, K14 G5NB, K15 G5NB, K16 G5NB, K17 G5NB, K2 G5NB, K3 G5NB, K4 G5NB, K5 G5NB, K6 G5NB, K7 G5NB, K8 G5NB, K9 G5NB, Q1 MMBT2222A, Q10 MMBT2222A, Q11 MMBT2222A, Q12 MMBT2222A, Q13 MMBT2222A, Q14 MMBT2222A, Q15 MMBT2222A, Q16 MMBT2222A, Q2 MMBT2222A, Q3 MMBT2222A, Q4 MMBT2222A, Q5 MMBT2222A, Q6 MMBT2222A, Q7 MMBT2222A, Q8 MMBT2222A, Q9 MMBT2222A, SW1 SW_Push, SW2 SW_Push, U1 URB2405YMD-10WR3, U10 LTV-817S, U11 LTV-817S, U12 LTV-817S, U13 LTV-817S, U14 LTV-817S, U15 LTV-817S, U16 LTV-817S, U17 LTV-817S, U18 LTV-817S, U19 LTV-817S, U2 AZ1117-3.3, U20 74HC138, U21 LTV-817S, U22 LTV-817S, U23 LTV-817S, U24 LTV-817S, U25 LTV-817S, U26 LTV-817S, U27 LTV-817S, U28 LTV-817S, U29 LTV-817S, U3 STM32F401R_B-C_Tx, U30 LTV-817S, U31 LTV-817S, U32 LTV-817S, U33 LTV-817S, U34 LTV-817S, U35 LTV-817S, U36 LTV-817S, U4 LTV-817S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

Commit message: modified:   DECON_Ctrl_Panel.kicad_pcb
Parts:
- added C38: 104, Capacitor_SMD:C_0805_2012Metric, B.Cu at (131.4, 144.9)
- added J1: Conn_01x02, TerminalBlock_MetzConnect:TerminalBlock_MetzConnect_Type086_RT03402HBLC_1x02_P3.81mm_Horizontal, F.Cu at (207.8, 168.3)
- C23, C24, C25, C26, C27, C28, C29, C30, C31, C32, C33, C34, C35, C36, C37: moved to B.Cu
- moved J18 171.7 mm to (117.0, 75.4)
- moved R129 166.9 mm to (264.0, 72.8), turned to -90 degrees
- moved R122 161.6 mm to (264.0, 66.4), turned to 90 degrees
- moved R128 154.3 mm to (255.8, 72.8), turned to -90 degrees
- moved Q16 154.0 mm to (260.0, 123.1)
- moved R121 153.0 mm to (255.8, 66.4), turned to 90 degrees
- moved R127 150.1 mm to (247.5, 72.8), turned to -90 degrees
- moved R120 148.3 mm to (247.5, 66.4), turned to 90 degrees
- moved D30 146.1 mm to (259.0, 114.8), turned to -90 degrees
- moved Q15 142.7 mm to (251.7, 123.1)
- moved Q13 141.1 mm to (235.2, 123.1)
- moved F1 140.7 mm to (121.7, 153.5)
- moved Q11 136.4 mm to (218.7, 123.1)
- moved D29 136.4 mm to (250.7, 114.8), turned to -90 degrees
- moved C7 135.5 mm to (97.4, 134.3), turned to 90 degrees
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Connections:
- K1 pad A1: Net-(D9-A) -> V_VALVE
- K1 pad A2: V_VALVE -> Net-(D9-A)
- K10 pad 14: RELAY_9 -> RELAY_8
- K10 pad A1: Net-(D24-A) -> V_VALVE
- K10 pad A2: V_VALVE -> Net-(D23-A)
- K11 pad 14: RELAY_10 -> RELAY_7
- K11 pad A1: Net-(D25-A) -> V_VALVE
- K11 pad A2: V_VALVE -> Net-(D22-A)
- K12 pad 14: RELAY_11 -> RELAY_6
- K12 pad A1: Net-(D26-A) -> V_VALVE
- K12 pad A2: V_VALVE -> Net-(D21-A)
- K13 pad A1: Net-(D31-A) -> V_VALVE
- K13 pad A2: V_VALVE -> Net-(D31-A)
- K14 pad A1: Net-(D32-A) -> V_VALVE
- K14 pad A2: V_VALVE -> Net-(D32-A)
- K15 pad A1: Net-(D33-A) -> V_VALVE
- K15 pad A2: V_VALVE -> Net-(D33-A)
- K16 pad A1: Net-(D34-A) -> V_VALVE
- K16 pad A2: V_VALVE -> Net-(D34-A)
- K17 pad 13: V_VALVE -> VBAT
- K17 pad 14: VBAT -> V_VALVE
- K2 pad A1: Net-(D10-A) -> V_VALVE
- K2 pad A2: V_VALVE -> Net-(D10-A)
- K3 pad A1: Net-(D11-A) -> V_VALVE
- K3 pad A2: V_VALVE -> Net-(D11-A)
- K4 pad A1: Net-(D12-A) -> V_VALVE
- K4 pad A2: V_VALVE -> Net-(D12-A)
- K5 pad A1: Net-(D13-A) -> V_VALVE
- K5 pad A2: V_VALVE -> Net-(D13-A)
- K6 pad A1: unconnected-(K6-PadA1) -> V_VALVE
- K6 pad A2: V_VALVE -> Net-(D14-A)
- K7 pad 14: RELAY_6 -> RELAY_11
- K7 pad A1: Net-(D21-A) -> V_VALVE
- K7 pad A2: V_VALVE -> Net-(D26-A)
- K8 pad 14: RELAY_7 -> RELAY_10
- K8 pad A1: Net-(D22-A) -> V_VALVE
- K8 pad A2: V_VALVE -> Net-(D25-A)
- K9 pad 14: RELAY_8 -> RELAY_9
- K9 pad A1: unconnected-(K9-PadA1) -> V_VALVE
- K9 pad A2: V_VALVE -> Net-(D24-A)
Routing:
- net V_VALVE: track 140.4 -> 53.0 mm
- net Net-(R71-Pad2): track 0.00 -> 9.57 mm
- net Net-(R43-Pad2): track 0.00 -> 9.57 mm
- net Net-(R42-Pad2): track 0.00 -> 9.57 mm
- net Net-(R13-Pad2): track 0.00 -> 9.57 mm
- net Net-(R73-Pad2): track 0.00 -> 9.57 mm
- net Net-(R72-Pad2): track 0.00 -> 9.57 mm
- net Net-(R70-Pad2): track 0.00 -> 9.57 mm
- net Net-(R47-Pad2): track 0.00 -> 9.57 mm
- net Net-(R46-Pad2): track 0.00 -> 9.57 mm
- net Net-(R45-Pad2): track 0.00 -> 9.57 mm
- net Net-(R44-Pad2): track 0.00 -> 9.57 mm
- net Net-(R17-Pad2): track 0.00 -> 9.57 mm
- net Net-(R16-Pad2): track 0.00 -> 9.57 mm
- net Net-(R15-Pad2): track 0.00 -> 9.57 mm
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
Commit message: modified:   DECON_Ctrl_Panel.kicad_pcb
Parts:
- removed the J1 at (207.8, 168.3)
- moved SW1 171.4 mm to (295.9, 93.5)
- moved SW2 158.4 mm to (283.5, 69.6)
- moved R122 146.5 mm to (126.9, 118.0), turned to -90 degrees
- moved R129 142.6 mm to (126.9, 111.7), turned to 90 degrees
- moved U36 137.0 mm to (130.8, 114.8), turned to 90 degrees
- moved C10 133.8 mm to (223.8, 98.4)
- moved C12 133.8 mm to (239.7, 96.7)
- moved C15 133.8 mm to (239.7, 93.7)
- moved C16 133.8 mm to (239.7, 90.7)
- moved C17 133.8 mm to (239.7, 87.7)
- moved C18 133.8 mm to (239.7, 84.7)
- moved C20 133.8 mm to (235.2, 96.7)
- moved J18 133.8 mm to (248.9, 97.5)
- moved J5 133.8 mm to (214.6, 97.6)
- moved C19 126.7 mm to (228.9, 94.5)
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Connections:
- C2 pad 1: MCU_EXTI -> MCU_BTN_4
- K17 pad 13: VBAT -> V_VALVE
- K17 pad 14: V_VALVE -> VBAT
- K17 pad A1: VBAT -> Net-(K17-PadA1)
- K17 pad A2: Net-(K17-PadA2) -> VBAT
- R2 pad 2: MCU_EXTI -> MCU_BTN_4
- R86 pad 2: Net-(K17-PadA2) -> Net-(K17-PadA1)
- SW1 pad 1: MCU_EXTI -> MCU_BTN_4
- U3 pad 10: MCU_RL2 -> MCU_A0
- U3 pad 11: MCU_RL3 -> MCU_SS_0
- U3 pad 14: MCU_RL4 -> MCU_SS_1
- U3 pad 15: MCU_RL5 -> MCU_EXTI
- U3 pad 16: MCU_RL6 -> MCU_RL0
- U3 pad 17: MCU_RL7 -> MCU_RL1
- U3 pad 20: MCU_RL8 -> MCU_RL2
- U3 pad 21: MCU_RL9 -> MCU_RL3
- U3 pad 22: MCU_RL10 -> MCU_RL4
- U3 pad 23: MCU_RL11 -> MCU_RL5
- U3 pad 24: MCU_RL12 -> MCU_RL6
- U3 pad 25: MCU_RL13 -> MCU_RL7
- U3 pad 26: MCU_RL14 -> MCU_RL8
- U3 pad 27: MCU_RL15 -> MCU_RL9
- U3 pad 28: MCU_SS_0 -> MCU_RL10
- U3 pad 29: MCU_SS_1 -> MCU_RL11
- U3 pad 30: unconnected-(U3-VCAP1-Pad30) -> VCAP1
- U3 pad 33: MCU_BTN_0 -> MCU_RL12
- U3 pad 34: MCU_BTN_1 -> MCU_RL13
- U3 pad 35: MCU_BTN_2 -> MCU_RL14
- U3 pad 36: MCU_BTN_3 -> MCU_RL15
- U3 pad 37: MCU_BTN_4 -> MCU_BTN_0
- U3 pad 38: MCU_A2 -> MCU_BTN_1
- U3 pad 39: MCU_A1 -> MCU_BTN_2
- U3 pad 40: MCU_A0 -> MCU_BTN_3
- U3 pad 41: MCU_EXTI -> MCU_BTN_4
- U3 pad 8: MCU_RL0 -> MCU_A2
- U3 pad 9: MCU_RL1 -> MCU_A1
Routing:
- net MCU_RL15: track 4.69 -> 77.7 mm
- net MCU_RL14: track 4.69 -> 69.8 mm
- net MCU_SS_1: track 0.00 -> 58.6 mm
- net MCU_RL13: track 4.69 -> 61.9 mm
- net GND_MCU: track 0.00 -> 56.0 mm
- net MCU_RL12: track 4.69 -> 53.9 mm
- net MCU_RL0: track 4.69 -> 47.6 mm
- net MCU_RL11: track 4.40 -> 46.1 mm
- net MCU_EXTI: track 0.00 -> 39.9 mm
- net 74138_Y7: track 0.00 -> 36.4 mm
- net MCU_RL1: track 4.69 -> 39.0 mm
- net MCU_RL10: track 4.69 -> 38.2 mm
- net MCU_RL2: track 4.71 -> 30.5 mm
- net MCU_RL9: track 4.69 -> 30.4 mm
- net 74138_Y6: track 0.00 -> 23.7 mm
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