File: relay.kicad_sch (KiCad schematic)
At the start: 129 parts, among them J24 Conn_01x10, K1 G5NB, K10 G5NB, K11 G5NB, K12 G5NB, K13 G5NB, K14 G5NB, K15 G5NB, K17 G5NB, K2 G5NB, K3 G5NB, K4 G5NB, K5 G5NB, K6 G5NB, K7 G5NB, K8 G5NB, K9 G5NB, Q1 MMBT2222A, Q10 MMBT2222A, Q11 MMBT2222A, Q12 MMBT2222A, Q13 MMBT2222A, Q14 MMBT2222A, Q15 MMBT2222A, Q17 MMBT2222A, Q2 MMBT2222A, Q3 MMBT2222A, Q4 MMBT2222A, Q5 MMBT2222A, Q6 MMBT2222A, Q7 MMBT2222A, Q8 MMBT2222A, Q9 MMBT2222A, U10 LTV-817S, U11 LTV-817S, U12 LTV-817S, U13 LTV-817S, U14 LTV-817S, U15 LTV-817S, U16 LTV-817S, U17 LTV-817S, U18 LTV-817S, U19 LTV-817S, U20 LTV-817S, U5 LTV-817S, U6 LTV-817S, U7 LTV-817S, U8 LTV-817S, U9 LTV-817S

Commit message: new file:   decon_ctrl.pdf
Parts:
- removed J24: Conn_01x10, Connector_Phoenix_MC:PhoenixContact_MC_1,5_10-G-3.81_1x10_P3.81mm_Horizontal, symbol Connector_Generic:Conn_01x10
Other:
- moved on the sheet: C10, C11, C12, C13, C14, C15, C16, C17, C18, C19, C20, C21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

Commit message: modified:   DECON_Ctrl_Panel.kicad_pcb
Parts:
- removed D10, D14, D18, D22, D26, D30, D6: 1N4148W, Diode_SMD:D_SOD-123, symbol Diode:1N4148W
- removed D13, D17, D21, D25, D29, D5, D9: LED, LED_SMD:LED_0805_2012Metric, symbol Device:LED
- added D10, D14, D18, D22, D26, D30, D6: LED, LED_SMD:LED_0805_2012Metric, symbol Device:LED
- added D13, D17, D21, D25, D29, D5, D9: 1N4148W, Diode_SMD:D_SOD-123, symbol Diode:1N4148W
- added R100, R101, R104, R105, R108, R32, R34, R36, R38, R41, R42, R63, R64, R81, R82, R85, R86: 10K, Resistor_SMD:R_0805_2012Metric, symbol Device:R
- added R102, R103, R106, R107, R35, R39, R40, R45, R46, R79, R80, R83, R84, R98, R99: 1K, Resistor_SMD:R_0805_2012Metric, symbol Device:R
- R10, R14, R18, R22, R26, R30, R6: value 510 -> 10K
- R11, R15, R19, R23, R27, R3, R31, R37, R7: value 510 -> 1K
- R13, R17, R2, R21, R25, R29, R5, R9: value 1K -> 10K
Connections:
- net 3.3V: now also R10.1, R11.1, R14.1, R15.1, R18.1, R19.1, R22.1, R23.1, R26.1, R27.1, R3.1, R30.1, R31.1, R6.1, R7.1, R101.1, R102.1, R105.1, R106.1, R32.1, R38.1, R39.1, R42.1, R45.1, R64.1, R79.1, R82.1, R83.1, R86.1, R98.1; no longer R12.1, R13.1, R16.1, R17.1, R20.1, R21.1, R24.1, R25.1, R28.1, R29.1, R4.1, R5.1, R8.1, R9.1
- net GND_VBAT: now also R13.2, R17.2, R21.2, R25.2, R29.2, R5.2, R9.2, R100.2, R104.2, R108.2, R34.2, R36.2, R41.2, R63.2, R81.2, R85.2
- net MCU_RL0: now also R32.2
- net MCU_RL1: now also R2.2
- net MCU_RL10: now also D22.1 (K), R64.2; no longer D24.1 (K)
- net MCU_RL11: now also D24.1 (K), R82.2
- net MCU_RL12: now also D20.1 (K), R42.2; no longer D12.1 (K)
- net MCU_RL13: now also D30.1 (K), R105.2
- net MCU_RL14: now also R101.2
- net MCU_RL15: now also D26.1 (K), R86.2
- net MCU_RL2: now also D4.1 (K), R6.2; no longer D16.1 (K)
- net MCU_RL3: now also R10.2, D6.1 (K)
- net MCU_RL4: now also D8.1 (K), R14.2; no longer D4.1 (K)
- net MCU_RL5: now also R18.2, D10.1 (K)
- net MCU_RL6: now also D12.1 (K), R22.2; no longer D20.1 (K)
- net MCU_RL7: now also R26.2, D14.1 (K)
- net MCU_RL8: now also D16.1 (K), R30.2; no longer D8.1 (K)
- net MCU_RL9: now also D18.1 (K), R38.2
- net RELAY_10: now also C19.1, K11.13; no longer C20.1, K12.13
- net RELAY_11: now also C20.1, K12.13; no longer C21.1, K13.13
- net RELAY_12: now also C18.1, K10.13; no longer C13.1, K6.13
- net RELAY_13: now also C23.1, K15.13; no longer C14.1, K7.13
- net RELAY_15: now also C21.1, K13.13; no longer C23.1, K15.13
- net RELAY_2: now also C9.1, K2.13; no longer C15.1, K8.13
- net RELAY_3: now also C10.1, K3.13; no longer C16.1, K9.13
- net RELAY_4: now also C11.1, K4.13; no longer C9.1, K2.13
- net RELAY_5: now also C12.1, K5.13; no longer C10.1, K3.13
- net RELAY_6: now also C13.1, K6.13; no longer C18.1, K10.13
- net RELAY_7: now also C14.1, K7.13; no longer C19.1, K11.13
- net RELAY_8: now also C15.1, K8.13; no longer C11.1, K4.13
- net RELAY_9: now also C16.1, K9.13; no longer C12.1, K5.13
- net VBAT: now also D13.1 (K), D17.1 (K), D21.1 (K), D25.1 (K), D29.1 (K), D5.1 (K), D9.1 (K)
- net at R4.2: now also Q1.1 (B), R5.1; no longer U6.1
- net at U5.1: now also R3.2; no longer R2.2
- net at K4.A2, Q4.3 (C): now also D9.2 (A)
- net at K6.A2, Q6.3 (C): now also D13.2 (A)
- net at U7.1: now also R11.2; no longer R5.2
- net at U7.2: now also D6.2 (A)
- net at U7.3: now also R12.1; no longer R7.1
- net at U15.2: now also D22.2 (A)
- net at R12.2: now also Q3.1 (B), R13.1; no longer U10.1
- net at U10.3: now also R24.1; no longer R14.1
- net at U12.3: now also R35.1; no longer R18.1
- net at Q8.1 (B): now also R35.2, R36.1; no longer R18.2
- net at Q13.1 (B): now also R100.1, R99.2; no longer R27.2
- net at U5.3: now also R4.1; no longer R3.1
- net at K2.A2, Q2.3 (C): now also D5.2 (A)
- net at R8.2: now also Q2.1 (B), R9.1; no longer U8.1
- net at K12.A2, Q12.3 (C): now also D25.2 (A)
- net at U11.1: now also R27.2; no longer R13.2
- net at U9.3: now also R20.1; no longer R11.1
- net at Q5.1 (B): now also R20.2, R21.1; no longer R11.2
- net at U20.1: now also R106.2; no longer R29.2
- net at U20.2: now also D30.2 (A)
- net at U20.3: now also R107.1; no longer R31.1
- net at Q4.1 (B): now also R16.2, R17.1; no longer R10.2
- net at U9.1: now also R19.2; no longer R9.2
- net at U11.3: now also R28.1; no longer R15.1
- net at Q7.1 (B): now also R28.2, R29.1; no longer R15.2
- net at U17.1: now also R98.2; no longer R25.2
- net at U17.2: now also D26.2 (A)
- net at U17.3: now also R99.1; no longer R27.1
- net at R24.2: now also Q6.1 (B), R25.1; no longer U16.1
- net at U16.3: now also R84.1; no longer R26.1
- net at Q10.1 (B): now also R46.2, R63.1; no longer R22.2
- net at K10.A2, Q10.3 (C): now also D21.2 (A)
- net at U15.1: now also R79.2; no longer R21.2
- net at U15.3: now also R80.1; no longer R23.1
- net at U14.1: now also R45.2; no longer R20.2
- net at R7.2: now also U6.1; no longer Q3.1 (B)
- net at K8.A2, Q8.3 (C): now also D17.2 (A)
- net at U19.3: now also R103.1; no longer R30.1
- net at Q14.1 (B): now also R103.2, R104.1; no longer R30.2
- net at Q12.1 (B): now also R84.2, R85.1; no longer R26.2
- net at K14.A2, Q14.3 (C): now also D29.2 (A)
- net at Q11.1 (B): now also R80.2, R81.1; no longer R23.2
- net at U6.3: now also R8.1; no longer R6.1
- net at U11.2: now also D14.2 (A)
- net at Q9.1 (B): now also R40.2, R41.1; no longer R19.2
- net at U13.1: now also R39.2; no longer R17.2
- net at U13.2: now also D18.2 (A)
- net at U13.3: now also R40.1; no longer R19.1
- net at Q15.1 (B): now also R107.2, R108.1; no longer R31.2
- net at U9.2: now also D10.2 (A)
- net at U19.1: now also R102.2; no longer R28.2
- net at Q17.1 (B), R37.2: now also R34.1
- net at U14.3: now also R46.1; no longer R22.1
- net at U12.1: now also R31.2; no longer R16.2
- net at U8.3: now also R16.1; no longer R10.1
- new net: R83.2, U16.1
- new net: R15.2, U8.1
- new net: R23.2, U10.1
Other:
- moved on the sheet: C17, D33, D37, K17, Q17, R33, R37, U18

Commit message: modified:   DECON_Ctrl_Panel.kicad_pcb
Parts:
- added K15: G5NB, Relay_THT:Relay_SPST_Omron_G5NB, symbol Relay:G5NB
- added R12, R13, R14, R27, R28, R29, R42, R43, R44, R57, R58, R59, R70, R71, R72, R81, R82: 470, Resistor_SMD:R_0805_2012Metric, symbol Device:R
- renumbered C18 to C22, C17 to C23, C13 to C24, C23 to C25, C8 to C26, C14 to C27, C22 to C28, C9 to C29, C15 to C30, C21 to C31, C10 to C32, C16 to C33, C11 to C34, C19 to C35, C12 to C36, C20 to C37, D3 to D10, D15 to D11, D30 to D12, D2 to D13, D29 to D15, D5 to D16, D28 to D18, D4 to D19, D16 to D20, D27 to D21, D7 to D22, D19 to D23, D26 to D24, D6 to D25, D18 to D26, D9 to D27, D23 to D28, D8 to D29, D21 to D3, D22 to D30, D11 to D31, D25 to D32, D10 to D33, D24 to D34, D37 to D4, D13 to D5, D20 to D6, D33 to D7, D12 to D8, D31 to D9, K10 to K1, K13 to K10, K3 to K11, K9 to K12, K4 to K13, K11 to K14, K5 to K16, K12 to K17, K17 to K2, K6 to K3, K15 to K4, K1 to K5, K7 to K6, K14 to K7, K2 to K8, K8 to K9, Q10 to Q1, Q13 to Q10, Q3 to Q11, Q9 to Q12, Q4 to Q13, Q11 to Q14, Q5 to Q15, Q12 to Q16, Q17 to Q2, Q6 to Q3, Q15 to Q4, Q1 to Q5, Q7 to Q6, Q14 to Q7, Q2 to Q8, Q8 to Q9, R22 to R10, R23 to R11, R46 to R15, R37 to R16, R24 to R17, R63 to R18, R34 to R19, R25 to R20, R105 to R21, R106 to R22, R2 to R23, R3 to R24, R26 to R25, R27 to R26, R107 to R30, R4 to R31, R28 to R32, R108 to R33, R5 to R34, R29 to R35, R101 to R36, R102 to R37, R6 to R38, R7 to R39, R30 to R40, R31 to R41, R103 to R45, R8 to R46, R35 to R47, R104 to R48, R9 to R49, R36 to R50, R86 to R51, R98 to R52, R10 to R53, R11 to R54, R38 to R55, R39 to R56, R42 to R6, R99 to R60, R12 to R61, R40 to R62, R100 to R63, R13 to R64, R41 to R65, R14 to R66, R15 to R67, R64 to R68, R79 to R69, R45 to R7, R16 to R73, R80 to R74, R17 to R75, R81 to R76, R18 to R77, R19 to R78, R82 to R79, R32 to R8, R83 to R80, R20 to R83, R21 to R85, R85 to R86, R33 to R9, U19 to U10, U6 to U11, U17 to U13, U7 to U14, U13 to U15, U8 to U16, U15 to U17, U9 to U18, U16 to U19, U14 to U4, U18 to U5, U10 to U6, U20 to U7, U5 to U8, U11 to U9
Connections:
- net VBAT: now also K15.14, K15.A1; no longer D10.1 (K), D11.1 (K), D15.1 (K), D16.1 (K), D17.1 (K), D21.1 (K), D22.1 (K), D23.1 (K), D27.1 (K), D28.1 (K), D3.1 (K), D31.1 (K), D4.1 (K), D5.1 (K), D9.1 (K), K1.14, K1.A1, K10.14, K10.A1, K11.14, K11.A1, K12.14, K12.A1, K13.14, K13.A1, K14.14, K14.A1, K16.14, K16.A1, K2.14, K2.A1, K3.14, K3.A1, K4.14, K4.A1, K5.14, K5.A1, K6.14, K6.A1, K7.14, K7.A1, K8.14, K8.A1, K9.14, K9.A1, U10.4, U11.4, U12.4, U13.4, U14.4, U15.4, U16.4, U17.4, U18.4, U4.4, U5.4, U6.4, U7.4, U8.4, U9.4
- net at D23.2 (A), Q12.3 (C): now also R59.1; no longer K12.A2
- net at D27.2 (A), Q13.3 (C): now also R70.1; no longer K13.A2
- net at D31.2 (A), Q15.3 (C): now also R81.1; no longer K16.A2
- net at D22.2 (A), Q11.3 (C): now also R58.1; no longer K11.A2
- net at D17.2 (A), Q9.3 (C): now also R44.1; no longer K9.A2
- net at D3.2 (A), Q1.3 (C): now also R12.1; no longer K1.A2
- net at D4.2 (A), Q2.3 (C): now also R13.1; no longer K2.A2
- net at D32.2 (A), Q16.3 (C): now also R82.1; no longer K17.A2
- net at D16.2 (A), Q8.3 (C): now also R43.1; no longer K8.A2
- net at D5.2 (A), Q3.3 (C): now also R14.1; no longer K3.A2
- net at D9.2 (A), Q4.3 (C): now also R27.1; no longer K4.A2
- net at D11.2 (A), Q6.3 (C): now also R29.1; no longer K6.A2
- net at D10.2 (A), Q5.3 (C): now also R28.1; no longer K5.A2
- net at D28.2 (A), Q14.3 (C): now also R71.1; no longer K14.A2
- net at D21.2 (A), Q10.3 (C): now also R57.1; no longer K10.A2
- net at D15.2 (A), Q7.3 (C): now also R42.1; no longer K7.A2
- new net: K3.A2, R14.2
- new net: K11.A2, R58.2
- new net: K9.A2, R44.2
- new net: K10.A2, R57.2
- new net: K2.A2, R13.2
- new net: K5.A2, R28.2
- new net: K8.A2, R43.2
- new net: K17.A2, R82.2
- new net: K7.A2, R42.2
- new net: K6.A2, R29.2
- new net: K16.A2, R81.2
- new net: K15.A2, R72.2
- new net: K14.A2, R71.2
- new net: K13.A2, R70.2
- new net: K12.A2, R59.2
- new net: K4.A2, R27.2
- new net: K1.A2, R12.2
- new net BUTTON_EN: R72.1
- new net V_VALVE: D10.1 (K), D11.1 (K), D15.1 (K), D16.1 (K), D17.1 (K), D21.1 (K), D22.1 (K), D23.1 (K), D27.1 (K), D28.1 (K), D3.1 (K), D31.1 (K), D4.1 (K), D5.1 (K), D9.1 (K), K1.14, K1.A1, K10.14, K10.A1, K11.14, K11.A1, K12.14, K12.A1, K13.14, K13.A1, K14.14, K14.A1, K15.13, K16.14, K16.A1, K2.14, K2.A1, K3.14, K3.A1, K4.14, K4.A1, K5.14, K5.A1, K6.14, K6.A1, K7.14, K7.A1, K8.14, K8.A1, K9.14, K9.A1, U10.4, U11.4, U12.4, U13.4, U14.4, U15.4, U16.4, U17.4, U18.4, U4.4, U5.4, U6.4, U7.4, U8.4, U9.4

Commit message: modified:   DECON_Ctrl_Panel.kicad_pcb
Parts:
- removed R12, R13, R14, R27, R28, R29, R42, R43, R44, R57, R58, R59, R70, R71, R81, R82: 470, Resistor_SMD:R_0805_2012Metric, symbol Device:R
- renumbered C23 to C22, C26 to C23, C29 to C24, C32 to C25, C34 to C26, C36 to C27, C24 to C28, C27 to C29, C33 to C31, C35 to C32, C37 to C33, C22 to C34, C25 to C35, C28 to C36, C31 to C37, D16 to D11, D22 to D12, D27 to D13, D31 to D14, D8 to D15, D14 to D16, D20 to D17, D26 to D18, D30 to D19, D34 to D20, D5 to D21, D11 to D22, D17 to D23, D23 to D24, D28 to D25, D32 to D26, D6 to D27, D12 to D28, D18 to D29, D7 to D3, D24 to D30, D3 to D31, D9 to D32, D15 to D33, D21 to D34, D13 to D4, D19 to D5, D25 to D6, D29 to D7, D33 to D8, D4 to D9, K2 to K1, K12 to K10, K14 to K11, K17 to K12, K1 to K13, K4 to K14, K7 to K15, K10 to K16, K15 to K17, K5 to K2, K8 to K3, K11 to K4, K13 to K5, K16 to K6, K3 to K7, K6 to K8, Q2 to Q1, Q12 to Q10, Q14 to Q11, Q16 to Q12, Q1 to Q13, Q4 to Q14, Q7 to Q15, Q10 to Q16, Q5 to Q2, Q8 to Q3, Q11 to Q4, Q13 to Q5, Q15 to Q6, Q3 to Q7, Q6 to Q8, R66 to R10, R77 to R11, R9 to R12, R24 to R13, R39 to R14, R54 to R15, R67 to R16, R78 to R17, R16 to R18, R31 to R19, R46 to R20, R61 to R21, R73 to R22, R83 to R23, R19 to R24, R34 to R25, R49 to R26, R64 to R27, R75 to R28, R85 to R29, R10 to R36, R25 to R37, R40 to R38, R55 to R39, R68 to R40, R79 to R41, R11 to R42, R26 to R43, R41 to R44, R56 to R45, R69 to R46, R80 to R47, R17 to R48, R32 to R49, R47 to R50, R62 to R51, R74 to R52, R84 to R53, R20 to R54, R35 to R55, R50 to R56, R65 to R57, R76 to R58, R86 to R59, R8 to R6, R6 to R66, R21 to R67, R36 to R68, R51 to R69, R23 to R7, R7 to R70, R22 to R71, R37 to R72, R52 to R73, R15 to R74, R30 to R75, R45 to R76, R60 to R77, R18 to R78, R33 to R79, R38 to R8, R48 to R80, R63 to R81, R72 to R86, R53 to R9, U6 to U10, U9 to U11, U15 to U13, U17 to U14, U19 to U15, U4 to U16, U7 to U17, U10 to U18, U13 to U19, U5 to U4, U8 to U5, U11 to U6, U14 to U7, U16 to U8, U18 to U9
Connections:
- net RELAY_0: now also K1.14; no longer K1.13
- net RELAY_1: now also K2.14; no longer K2.13
- net RELAY_10: now also K11.14; no longer K11.13
- net RELAY_11: now also K12.14; no longer K12.13
- net RELAY_12: now also K13.14; no longer K13.13
- net RELAY_13: now also K14.14; no longer K14.13
- net RELAY_14: now also K15.14; no longer K15.13
- net RELAY_15: now also K16.14; no longer K16.13
- net RELAY_2: now also K3.14; no longer K3.13
- net RELAY_3: now also K4.14; no longer K4.13
- net RELAY_4: now also K5.14; no longer K5.13
- net RELAY_5: now also K6.14; no longer K6.13
- net RELAY_6: now also K7.14; no longer K7.13
- net RELAY_7: now also K8.14; no longer K8.13
- net RELAY_8: now also K9.14; no longer K9.13
- net RELAY_9: now also K10.14; no longer K10.13
- net VBAT: no longer D26.1 (K), K12.14, K12.A1, U15.4
- net V_VALVE: now also D26.1 (K), K1.13, K1.A2, K10.13, K10.A2, K11.13, K11.A2, K12.13, K12.A2, K13.13, K13.A2, K14.13, K14.A2, K15.13, K15.A2, K16.13, K16.A2, K2.13, K2.A2, K3.13, K3.A2, K4.13, K4.A2, K5.13, K5.A2, K6.13, K6.A2, K7.13, K7.A2, K8.13, K8.A2, K9.13, K9.A2, U15.4; no longer K1.14, K1.A1, K10.14, K10.A1, K11.14, K11.A1, K13.14, K13.A1, K14.14, K14.A1, K15.14, K15.A1, K16.14, K16.A1, K2.14, K2.A1, K3.14, K3.A1, K4.14, K4.A1, K5.14, K5.A1, K6.14, K6.A1, K7.14, K7.A1, K8.14, K8.A1, K9.14, K9.A1
- net at D24.2 (A), Q10.3 (C): now also K10.A1
- net at D13.2 (A), Q5.3 (C): now also K5.A1
- net at D21.2 (A), Q7.3 (C): now also K7.A1
- net at D34.2 (A), Q16.3 (C): now also K16.A1
- net at D31.2 (A), Q13.3 (C): now also K13.A1
- net at D10.2 (A), Q2.3 (C): now also K2.A1
- net at D12.2 (A), Q4.3 (C): now also K4.A1
- net at D26.2 (A), Q12.3 (C): now also K12.A1
- net at D32.2 (A), Q14.3 (C): now also K14.A1
- net at D11.2 (A), Q3.3 (C): now also K3.A1
- net at D22.2 (A), Q8.3 (C): now also K8.A1
- net at D33.2 (A), Q15.3 (C): now also K15.A1
- net at D25.2 (A), Q11.3 (C): now also K11.A1
- net at D9.2 (A), Q1.3 (C): now also K1.A1
Other:
- moved on the sheet: C22, C23, C24, C25, C26, C27, C28, C29, C30, C31, C32, C33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

Commit message: modified:   DECON_Ctrl_Panel.kicad_pcb
Parts:
- removed K1, K10, K11, K12, K13, K14, K15, K16, K17, K2, K3, K4, K5, K6, K7, K8, K9: G5NB, Relay_THT:Relay_SPST_Omron_G5NB, symbol Relay:G5NB
- added C38: 104, Capacitor_SMD:C_0805_2012Metric, symbol Device:C
- added K1, K10, K11, K12, K13, K14, K15, K16, K17, K2, K3, K4, K5, K6, K7, K8, K9: G5NB, Relay_THT:Relay_SPST_Omron_G5NB, symbol Son_KiCad_lib:G5NB
Connections:
- net GND_VBAT: now also C38.2
- net RELAY_0: now also K1.14
- net RELAY_1: now also K2.14
- net RELAY_10: now also K8.14
- net RELAY_11: now also K7.14
- net RELAY_12: now also K13.14
- net RELAY_13: now also K14.14
- net RELAY_14: now also K15.14
- net RELAY_15: now also K16.14
- net RELAY_2: now also K3.14
- net RELAY_3: now also K4.14
- net RELAY_4: now also K5.14
- net RELAY_5: now also K6.14
- net RELAY_6: now also K12.14
- net RELAY_7: now also K11.14
- net RELAY_8: now also K10.14
- net RELAY_9: now also K9.14
- net VBAT: now also K17.13, K17.A1
- net V_VALVE: now also C38.1, K1.13, K1.A1, K10.13, K10.A1, K11.13, K11.A1, K12.13, K12.A1, K13.13, K13.A1, K14.13, K14.A1, K15.13, K15.A1, K16.13, K16.A1, K17.14, K2.13, K2.A1, K3.13, K3.A1, K4.13, K4.A1, K5.13, K5.A1, K6.13, K6.A1, K7.13, K7.A1, K8.13, K8.A1, K9.13, K9.A1
- net at D24.2 (A), Q10.3 (C): now also K9.A2
- net at D13.2 (A), Q5.3 (C): now also K5.A2
- net at D14.2 (A), Q6.3 (C): now also K6.A2
- net at D12.2 (A), Q4.3 (C): now also K4.A2
- net at D23.2 (A), Q9.3 (C): now also K10.A2
- net at D31.2 (A), Q13.3 (C): now also K13.A2
- net at D9.2 (A), Q1.3 (C): now also K1.A2
- net at D26.2 (A), Q12.3 (C): now also K7.A2
- net at D11.2 (A), Q3.3 (C): now also K3.A2
- net at D21.2 (A), Q7.3 (C): now also K12.A2
- net at D32.2 (A), Q14.3 (C): now also K14.A2
- net at D22.2 (A), Q8.3 (C): now also K11.A2
- net at D10.2 (A), Q2.3 (C): now also K2.A2
- net at D25.2 (A), Q11.3 (C): now also K8.A2
- net at R86.2: now also K17.A2
- net at D34.2 (A), Q16.3 (C): now also K16.A2
- net at D33.2 (A), Q15.3 (C): now also K15.A2

Commit message: modified:   DECON_Ctrl_Panel.kicad_pcb
Connections:
- net VBAT: now also K17.14, K17.A2; no longer K17.13, K17.A1
- net V_VALVE: now also K17.13; no longer K17.14
- net at R86.2: now also K17.A1; no longer K17.A2
Other:
- moved on the sheet: C38
Changed lines of the file:
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@@
 	)
 	(junction
-		(at 339.09 215.9)
+		(at 336.55 215.9)
 		(diameter 0)
 		(color 0 0 0 0)
@@
 	(wire
 		(pts
-			(xy 326.39 198.12) (xy 336.55 198.12)
+			(xy 326.39 198.12) (xy 339.09 198.12)
 		)
 		(stroke
@@
 	(wire
 		(pts
+			(xy 339.09 198.12) (xy 339.09 199.39)
+		)
+		(stroke
+			(width 0)
+			(type default)
+		)
+	)
+	(wire
+		(pts
 			(xy 29.21 177.8) (xy 31.75 177.8)
 		)
@@
 	(wire
 		(pts
-			(xy 339.09 223.52) (xy 339.09 224.79)
+			(xy 336.55 223.52) (xy 336.55 224.79)
 		)
 		(stroke
@@
 	(wire
 		(pts
-			(xy 340.36 224.79) (xy 339.09 224.79)
+			(xy 337.82 224.79) (xy 336.55 224.79)
 		)
 		(stroke
@@
 	(wire
 		(pts
-			(xy 340.36 215.9) (xy 339.09 215.9)
+			(xy 337.82 215.9) (xy 336.55 215.9)
 		)
 		(stroke
@@
 	(wire
 		(pts
-			(xy 339.09 215.9) (xy 339.09 214.63)
+			(xy 336.55 215.9) (xy 336.55 214.63)
 		)
 		(stroke
@@
 	(wire
 		(pts
-			(xy 336.55 198.12) (xy 336.55 199.39)
-		)
-		(stroke
-			(width 0)
-			(type default)
-		)
-	)
-	(wire
-		(pts
 			(xy 156.21 172.72) (xy 153.67 172.72)
 		)
@@
 	(global_label "V_VALVE"
 		(shape input)
-		(at 340.36 215.9 0)
+		(at 337.82 215.9 0)
 		(fields_autoplaced yes)
 		(effects
@@
 		)
 		(property "Intersheetrefs" "${INTERSHEET_REFS}"
-			(at 350.8443 215.9 0)
+			(at 348.3043 215.9 0)
 			(effects
 				(font
@@
 	(global_label "GND_VBAT"
 		(shape input)
-		(at 340.36 224.79 0)
+		(at 337.82 224.79 0)
 		(fields_autoplaced yes)
 		(effects
@@
 		)
 		(property "Intersheetrefs" "${INTERSHEET_REFS}"
-			(at 352.5981 224.79 0)
+			(at 350.0581 224.79 0)
 			(effects
 				(font
@@
 	(symbol
 		(lib_id "Device:C")
-		(at 339.09 219.71 0)
+		(at 336.55 219.71 0)
 		(unit 1)
 		(exclude_from_sim no)
@@
 		(fields_autoplaced yes)
 		(property "Reference" "C38"
-			(at 342.9 218.4399 0)
+			(at 340.36 218.4399 0)
 			(effects
 				(font
@@
 		)
 		(property "Value" "104"
-			(at 342.9 220.9799 0)
+			(at 340.36 220.9799 0)
 			(effects
 				(font
@@
 		)
 		(property "Footprint" "Capacitor_SMD:C_0805_2012Metric"
-			(at 340.0552 223.52 0)
+			(at 337.5152 223.52 0)
 			(effects
 				(font
@@
 		)
 		(property "Datasheet" "~"
-			(at 339.09 219.71 0)
+			(at 336.55 219.71 0)
 			(effects
 				(font
@@
 		)
 		(property "Description" "Unpolarized capacitor"
-			(at 339.09 219.71 0)
+			(at 336.55 219.71 0)
 			(effects
 				(font
@@
 		(lib_id "Son_KiCad_lib:G5NB")
 		(at 331.47 207.01 0)
-		(mirror x)
 		(unit 1)
 		(exclude_from_sim no)
@@
 		(dnp no)
 		(property "Reference" "K17"
-			(at 342.9 208.2801 0)
+			(at 342.9 205.7399 0)
 			(effects
 				(font
@@
 		)
 		(property "Value" "G5NB"
-			(at 342.9 205.7401 0)
+			(at 342.9 208.2799 0)
 			(effects
 				(font
@@
 		)
 		(property "Footprint" "Relay_THT:Relay_SPST_Omron_G5NB"
-			(at 342.9 205.74 0)
+			(at 342.9 208.28 0)
 			(effects
 				(font
@@
 		)
 		(property "Datasheet" "https://omronfs.omron.com/en_US/ecb/products/pdf/en-g5nb_el.pdf"
-			(at 342.9 203.2 0)
+			(at 342.9 210.82 0)
 			(effects
 				(font
